File: photon_bldc/hardware/pcb/photon_bldc/photon_bldc.kicad_pcb (KiCad board)
At the start: 4 copper layers, 165 x 60 mm, 54 parts, among them J1 Conn_01x17, SW1 SW_DPDT_x2, U1 STM32G474RBTx, U2 LM1117MP-5.0, U3 LM1117MP-3.3, U4 HC-04S, X1 32.768KHz, Y1 Crystal_GND24

Commit message: Small updates to PCB
Parts:
- moved C6 1.70 mm to (209.9, 119.3)
Routing:
- net GND: track 83.1 -> 84.2 mm
Changed lines of the file:
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@@
 		)
 		(fp_text user "${REFERENCE}"
-			(at 0 0 360)
+			(at 0 0 0)
 			(layer "F.Fab")
 			(effects
@@
 		)
 		(fp_circle
-			(center -7.2998 -5.3001)
-			(end -7.0999 -5.3001)
-			(stroke
-				(width 0.4)
-				(type default)
-			)
-			(fill none)
-			(layer "Dwgs.User")
-		)
-		(fp_circle
 			(center -6.5 -12.25)
 			(end -6.47 -12.25)
@@
 		(tags "LED")
 		(property "Reference" "D2"
-			(at 0 -1.43 360)
+			(at 0 -1.43 0)
 			(layer "F.SilkS")
 			(hide yes)
@@
 		)
 		(property "Value" "LED"
-			(at 0 1.43 360)
+			(at 0 1.43 0)
 			(layer "F.Fab")
 			(hide yes)
@@
 		)
 		(fp_text user "${REFERENCE}"
-			(at 0 0 360)
+			(at 0 0 0)
 			(layer "F.Fab")
 			(effects
@@
 		(tags "inductor")
 		(property "Reference" "L1"
-			(at 2.3125 0 360)
+			(at 2.3125 0 0)
 			(layer "B.SilkS")
 			(effects
@@
 		)
 		(property "Value" "27nH"
-			(at 0 -1.43 360)
+			(at 0 -1.43 0)
 			(layer "B.Fab")
 			(effects
@@
 		)
 		(fp_text user "${REFERENCE}"
-			(at 0 0 360)
+			(at 0 0 0)
 			(layer "B.Fab")
 			(effects
@@
 		(tags "capacitor")
 		(property "Reference" "C8"
-			(at 2.5 0 360)
+			(at 2.5 0 0)
 			(layer "B.SilkS")
 			(effects
@@
 		)
 		(property "Value" "100n"
-			(at 0 -1.43 360)
+			(at 0 -1.43 0)
 			(layer "B.Fab")
 			(effects
@@
 		)
 		(fp_text user "${REFERENCE}"
-			(at 0 0 360)
+			(at 0 0 0)
 			(layer "B.Fab")
 			(effects
@@
 		(tags "capacitor")
 		(property "Reference" "C4"
-			(at 0 1.43 360)
+			(at 0 1.43 0)
 			(layer "B.SilkS")
 			(effects
@@
 		)
 		(property "Value" "100n"
-			(at 0 -1.43 360)
+			(at 0 -1.43 0)
 			(layer "B.Fab")
 			(effects
@@
 		)
 		(fp_text user "${REFERENCE}"
-			(at 0 0 360)
+			(at 0 0 0)
 			(layer "B.Fab")
 			(effects
@@
 		(tags "SMD SMT crystal")
 		(property "Reference" "Y1"
-			(at -0.2 -1.95 360)
+			(at -0.2 -1.95 0)
 			(layer "B.SilkS")
 			(effects
@@
 		)
 		(property "Value" "Crystal_GND24"
-			(at 0 -2 360)
+			(at 0 -2 0)
 			(layer "B.Fab")
 			(hide yes)
@@
 		)
 		(fp_text user "${REFERENCE}"
-			(at 0 0 360)
+			(at 0 0 0)
 			(layer "B.Fab")
 			(effects
@@
 		(tags "capacitor")
 		(property "Reference" "R1"
-			(at 0 1.43 360)
+			(at 0 1.43 0)
 			(layer "B.SilkS")
 			(effects
@@
 		)
 		(property "Value" "510"
-			(at 0 -1.43 360)
+			(at 0 -1.43 0)
 			(layer "B.Fab")
 			(effects
@@
 		)
 		(fp_text user "${REFERENCE}"
-			(at 0 0 360)
+			(at 0 0 0)
 			(layer "B.Fab")
 			(effects
@@
 		(tags "capacitor")
 		(property "Reference" "C1"
-			(at -2.775 0 360)
+			(at -2.775 0 0)
 			(layer "B.SilkS")
 			(effects
@@
 		)
 		(property "Value" "4u7"
-			(at 0 -1.43 360)
+			(at 0 -1.43 0)
 			(layer "B.Fab")
 			(effects
@@
 		)
 		(fp_text user "${REFERENCE}"
-			(at 0 0 360)
+			(at 0 0 0)
 			(layer "B.Fab")
 			(effects
@@
 	(footprint "Capacitor_SMD:C_0603_1608Metric"
 		(layer "B.Cu")
-		(at 210 121)
+		(at 209.9 119.3)
 		(descr "Capacitor SMD 0603 (1608 Metric), square (rectangular) end terminal, IPC_7351 nominal, (Body size source: IPC-SM-782 page 76, https://www.pcb-3d.com/wordpress/wp-content/uploads/ipc-sm-782a_amendment_1_and_2.pdf), generated with kicad-footprint-generator")
 		(tags "capacitor")
 		(property "Reference" "C6"
-			(at 0 1.43 360)
+			(at 0 1.43 0)
 			(layer "B.SilkS")
 			(effects
@@
 		)
 		(property "Value" "100n"
-			(at 0 -1.43 360)
+			(at 0 -1.43 0)
 			(layer "B.Fab")
 			(effects
@@
 		)
 		(fp_text user "${REFERENCE}"
-			(at 0 0 360)
+			(at 0 0 0)
 			(layer "B.Fab")
 			(effects
@@
 		(tags "capacitor")
 		(property "Reference" "C9"
-			(at -2.775 0 360)
+			(at -2.775 0 0)
 			(layer "B.SilkS")
 			(effects
@@
 		)
 		(property "Value" "100n"
-			(at 0 -1.43 360)
+			(at 0 -1.43 0)
 			(layer "B.Fab")
 			(effects
@@
 		)
 		(fp_text user "${REFERENCE}"
-			(at 0 0 360)
+			(at 0 0 0)
 			(layer "B.Fab")
 			(effects
@@
 		(tags "resistor")
 		(property "Reference" "R7"
-			(at 0 1.43 360)
+			(at 0 1.43 0)
 			(layer "B.SilkS")
 			(effects
@@
 		)
 		(property "Value" "100R"
-			(at 0 -1.43 360)
+			(at 0 -1.43 0)
 			(layer "B.Fab")
 			(effects
@@
 		)
 		(fp_text user "${REFERENCE}"
-			(at 0 0 360)
+			(at 0 0 0)
 			(layer "B.Fab")
 			(effects
@@
 	)
 	(segment
-		(start 197.2501 87.2501)
-		(end 196.7 86.7)
+		(start 204.4 120.6)
+		(end 203.1 121.9)
 		(width 0.3)
 		(layer "F.Cu")
@@
 	)
 	(segment
-		(start 203.1 122.8)
-		(end 204.5 121.4)
+		(start 203.1 121.9)
+		(end 203.1 123)
 		(width 0.3)
 		(layer "F.Cu")
@@
 	)
 	(segment
-		(start 213.23 98.4)
-		(end 213.23 100.63)
+		(start 197.2501 87.2501)
+		(end 196.7 86.7)
 		(width 0.3)
 		(layer "F.Cu")
@@
 	)
 	(segment
-		(start 196.7 86.7)
-		(end 196.6 86.6)
+		(start 213.23 98.4)
+		(end 213.23 100.63)
 		(width 0.3)
 		(layer "F.Cu")
@@
 	)
 	(segment
-		(start 203.1 123)
-		(end 203.1 122.8)
+		(start 196.7 86.7)
+		(end 196.6 86.6)
 		(width 0.3)
 		(layer "F.Cu")
@@
 	)
 	(via
-		(at 204.5 121.4)
+		(at 204.4 120.6)
 		(size 0.7)
 		(drill 0.3)
@@
 	)
 	(segment
+		(start 204.4 120.6)
+		(end 205.7 119.3)
+		(width 0.3)
+		(layer "B.Cu")
+		(net 1)
+	)
+	(segment
 		(start 166.5 73.7)
 		(end 168.4 73.7)
@@
 	)
 	(segment
+		(start 205.7 119.3)
+		(end 209.125 119.3)
+		(width 0.3)
+		(layer "B.Cu")
+		(net 1)
+	)
+	(segment
 		(start 140.1 91.2)
 		(end 139.4 91.2)
@@
 	)
 	(segment
-		(start 204.9 121)
-		(end 204.5 121.4)
-		(width 0.3)
-		(layer "B.Cu")
-		(net 1)
-	)
-	(segment
 		(start 181.425 105.1)
 		(end 181.425 104.325)
@@
 	)
 	(segment
-		(start 209.225 121)
-		(end 204.9 121)
-		(width 0.3)
-		(layer "B.Cu")
-		(net 1)
-	)
-	(segment
 		(start 178.75 100.6)
 		(end 178.75 99.175)
@@
 	)
 	(segment
-		(start 210.9 121.9)
-		(end 210.9 121.8)
-		(width 0.3)
-		(layer "F.Cu")
-		(net 4)
-	)
-	(segment
-		(start 210.9 123)
-		(end 210.9 121.9)
-		(width 0.3)
-		(layer "F.Cu")
-		(net 4)
-	)
-	(segment
 		(start 215.77 95.5)
 		(end 214.47 96.8)
@@
 	)
 	(segment
+		(start 210.775 122.875)
+		(end 210.775 121.2)
+		(width 0.3)
+		(layer "F.Cu")
+		(net 4)
+	)
+	(segment
 		(start 215.77 94.5)
 		(end 215.77 95.5)
@@
 	)
 	(via
-		(at 210.9 121.9)
+		(at 210.775 121.2)
 		(size 0.7)
 		(drill 0.3)
@@
 	)
 	(segment
-		(start 210.775 121)
-		(end 210.775 121.775)
+		(start 210.775 121.2)
+		(end 210.775 103.175)
 		(width 0.3)
 		(layer "B.Cu")
@@
 	)
 	(segment
-		(start 210.775 121.775)
-		(end 210.9 121.9)
-		(width 0.3)
-		(layer "B.Cu")
-		(net 4)
-	)
-	(segment
 		(start 210.775 103.175)
 		(end 205.4 97.8)
@@
 	)
 	(segment
-		(start 210.775 121)
-		(end 210.775 103.175)
-		(width 0.3)
-		(layer "B.Cu")
-		(net 4)
-	)
-	(segment
 		(start 181.45 102.35)
 		(end 181.5 102.4)
@@
 		(hatch edge 0.5)
 		(priority 2)
-		(connect_pads
+		(connect_pads yes
 			(clearance 0.5)
 		)

Commit message: g071
Parts:
- removed PROG2: Conn_02x07_Odd_Even, Connector_PinHeader_1.27mm:PinHeader_2x07_P1.27mm_Vertical_SMD
- removed R7: 100R, Resistor_SMD:R_0603_1608Metric
- added PROG1: Conn_02x07_Odd_Even, Connector_PinHeader_1.27mm:PinHeader_2x07_P1.27mm_Vertical_SMD, F.Cu at (213.2, 96.5)
- added R5: 100R, Resistor_SMD:R_0603_1608Metric, B.Cu at (214.5, 102.1)
Connections:
- U1 pad 56: PB3 -> SYS_JTDO_SWO
Routing:
- net SYS_JTDO_SWO: track 0.00 -> 30.9 mm, vias 0 -> 1
- net Net-(PROG1-Pin_11): track 0.00 -> 3.88 mm, vias 0 -> 1
- net Net-(PROG2-Pin_11): track 3.78 -> 0.00 mm, vias 1 -> 0
- net +3.3V: track 37.7 -> 38.2 mm, vias 3 -> 2
Other:
- board text added: "PHOTON"
- board text removed: "-"
