File: photon_bldc/hardware/pcb/G31_ESC/ESC_PCB/ESC_PCB.kicad_sch (KiCad schematic)
At the start: 21 parts, among them J1 PWM_Input, J2 Motor_Plus, J3 Motor_Minus, J4 Conn_01x08, U1 STM32G431K6Ux, U2 AMS1117-5.0, U3 AMS1117-3.3, U4 74AHC1G86, U5 74AHC1G86

Commit message: g071
Parts:
- removed C10: 100n, Capacitor_SMD:C_0603_1608Metric, symbol Device:C
- removed C11: 1u, Capacitor_SMD:C_0603_1608Metric, symbol Device:C
- removed L1: 27n, Inductor_SMD:L_0603_1608Metric, symbol Device:L
- removed U1: STM32G431K6Ux, Package_DFN_QFN:QFN-32-1EP_5x5mm_P0.5mm_EP3.45x3.45mm, symbol MCU_ST_STM32G4:STM32G431K6Ux
- added R2: 10k, symbol Device:R
- added U1: STM32G071GBUx, Package_DFN_QFN:QFN-28_4x4mm_P0.5mm, symbol MCU_ST_STM32G0:STM32G071GBUx
- C5: value 4u7 -> 100nF; footprint Capacitor_SMD:C_0603_1608Metric -> (none)
- C6: value 100n -> 4.7uF; footprint Capacitor_SMD:C_0603_1608Metric -> (none)
- C7: value 100n -> 100nF; footprint Capacitor_SMD:C_0603_1608Metric -> (none)
Connections:
- net +3V3: now also R2.1; no longer C5.1
- net GND: now also U1.4 (VSS)
- net PA0: now also U1.6 (PA0)
- net PA1: now also U1.7 (PA1)
- net PA10: now also U1.19 (PA12/PA10)
- net PA2: now also U1.8 (PA2)
- net PA3: now also U1.9 (PA3)
- net PA7: now also U1.13 (PA7)
- net PA9: now also U1.18 (PA11/PA9)
- net PB0: now also U1.14 (PB0)
- net PB4: now also U1.24 (PB4)
- net PB6: now also U1.26 (PB6)
- new net: C5.1, R2.2, U1.5 (PF2)
- new net +3.3V: U1.3 (VDD)
- new net PB1: U1.15 (PB1)
- new net PB7: U1.27 (PB7)
- new net PB8: U1.28 (PB8)
- new net SWCLK: U1.21 (PA14)
- new net SWDIO: U1.20 (PA13)
- no-connect marks 0 -> 9
Other:
- note added: "STM32G071GBU6"
- note removed: "STM32G431"

Commit message: ESC schemat continued
Parts:
- added C10, C11, C9: 1uF, symbol Device:C
- added D1, D2, D3: D, symbol Device:D
- added Q1, Q2, Q3, Q4, Q5, Q6: NMOS, symbol Simulation_SPICE:NMOS
- added U6: ~, Fortior Tech FD6288Q driver library:QFN50P400X400X90-25N, symbol ESC library:FD6288Q
Connections:
- net GND: now also Q4.3 (S), Q5.3 (S), Q6.3 (S), U6.6 (COM)
- net VDC: now also Q1.1 (D), Q2.1 (D), Q3.1 (D)
- new net: C9.1, D1.1 (K), U6.20 (VB1)
- new net: C9.2, U6.18 (VS1)
- new net: C11.2, U6.12 (VS3)
- new net: C11.1, D3.1 (K), U6.14 (VB3)
- new net: C10.2, U6.15 (VS2)
- new net: C10.1, D2.1 (K), U6.17 (VB2)
- new net +8V: D1.2 (A), D2.2 (A), D3.2 (A), U6.4 (VCC)
- new net A: Q1.3 (S), Q4.1 (D)
- new net B: Q3.3 (S), Q5.1 (D)
- new net C: Q2.3 (S), Q6.1 (D)
- new net GHA: Q1.2 (G), U6.22 (HIN1)
- new net GHB: Q3.2 (G), U6.23 (HIN2)
- new net GHC: Q2.2 (G), U6.24 (HIN3)
- new net GLA: Q4.2 (G), U6.1 (LIN1)
- new net GLB: Q5.2 (G), U6.2 (LIN2)
- new net GLC: Q6.2 (G), U6.3 (LIN3)
- no-connect marks 9 -> 12
Other:
- moved on the sheet: C1, C2, C3, C4, C5, C6, C7, C8, J1, J2, J3, J4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

Commit message: 0.0
Parts:
- removed C8: C, symbol Device:C
- removed J1: PWM_Input, symbol Connector_Generic:Conn_01x02
- removed J4: Conn_01x08, symbol Connector_Generic:Conn_01x08
- removed R1: 10K, symbol Device:R
- removed U4, U5: 74AHC1G86, symbol 74xGxx:74AHC1G86
Connections:
- net +8V is gone; now on net +3V3: D1.2 (A), D2.2 (A), D3.2 (A), U6.4 (VCC)
- net PB7 is gone; now on net BEMF_REF: U1.27 (PB7)
- net GHA: now also U6.19 (HO1); no longer U6.22 (HIN1)
- net GHB: now also U6.16 (HO2); no longer U6.23 (HIN2)
- net GHC: now also U6.13 (HO3); no longer U6.24 (HIN3)
- net GLA: now also U6.11 (LO1); no longer U6.1 (LIN1)
- net GLB: now also U6.10 (LO2); no longer U6.2 (LIN2)
- net GLC: now also U6.9 (LO3); no longer U6.3 (LIN3)
- net HA: now reaches U1.16 (PA8)
- net HA: now also U6.22 (HIN1)
- net PA0 renamed BEMF_REF
- net PA1 renamed BEMF_A
- net PA10 renamed HC
- net HC: now also U6.24 (HIN3)
- net PA3 renamed BEMF_B
- net PA7: no longer names the net of U1.13 (PA7)
- net PA9 renamed HB
- net HB: now also U6.23 (HIN2)
- net PB0 renamed LB
- net LB: now also U6.2 (LIN2)
- net PB1 renamed LC
- net LC: now also U6.3 (LIN3)
- net PB4 renamed BEMF_C
- new net LA: U6.1 (LIN1)
Other:
- note added: "Mosfet Driver"
- moved on the sheet: C5, Q1, Q2, Q3, Q4, Q5, Q6, R2, U1

Commit message: gg
Parts:
- added C12: 100nF, symbol Device:C
- added C8: 100uF, symbol Device:C
- added R1, R5, R8: 33K, symbol Device:R
- added R10, R3, R7: 10K, symbol Device:R
- added R4, R6, R9: 3.3K, symbol Device:R
Connections:
- net +3.3V: now also C12.1, C8.1
- net BEMF_A: now also R1.2, R3.1, R4.1
- net BEMF_B: now also R5.2, R6.1, R7.1
- net BEMF_C: now also R10.1, R8.2, R9.1
- net BEMF_REF: now also R10.2, R3.2, R7.2
- net GND: now also C12.2, C8.2, R4.2, R6.2, R9.2
- net A renamed PHASE_A
- net PHASE_A: now also R1.1
- net B renamed PHASE_B
- net PHASE_B: now also R5.1
- net C renamed PHASE_C
- net PHASE_C: now also R8.1

Commit message: jjjju
Parts:
- added C13, C14, C15, C16, C17, C18, C19, C20, C21, C22, C23, C24, C25, C26, C27, C28, C29, C30, C31, C32: 10uF, symbol Device:C
- added D4: LED, LED_SMD:LED_0603_1608Metric, symbol Device:LED
- added J1: Conn_01x03, symbol Connector_Generic:Conn_01x03
- added R11: 510, Capacitor_SMD:C_0603_1608Metric, symbol Device:R
- C10, C11, C9: value 1uF -> 4.7uF
- C8: value 100uF -> 10uF
Connections:
- net +3.3V: now also D4.2 (A)
- net GND: now also C13.2, C14.2, C15.2, C16.2, C17.2, C18.2, C19.2, C20.2, C21.2, C22.2, C23.2, C24.2, C25.2, C26.2, C27.2, C28.2, C29.2, C30.2, C31.2, C32.2, R11.2
- net PA2 renamed INPUT
- new net: D4.1 (K), R11.1
- new net VCC: C13.1, C14.1, C15.1, C16.1, C17.1, C18.1, C19.1, C20.1, C21.1, C22.1, C23.1, C24.1, C25.1, C26.1, C27.1, C28.1, C29.1, C30.1, C31.1, C32.1
Other:
- note removed: "1A LOW DROPOUT VOLTAGE REGULATORS"
- moved on the sheet: C10, C11, C12, C6, C7, C8, C9, D1, D2, D3, J2, J3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

Commit message: Mosfet footprints Added
Parts:
- C10, C11, C9: value 4.7uF -> 10uF
- C5, C6, C7: footprint (none) -> Capacitor_SMD:C_0603_1608Metric
- D1, D2, D3: footprint (none) -> Diode_SMD:D_SOD-523
- Q1, Q2, Q3, Q4, Q5, Q6: footprint (none) -> Fortior Tech FD6288Q driver library:TSON-8(3.1x3.1)
- renumbered J1 to RC_Connector1
Connections:
- net GND: now also RC_Connector1.1 (Pin_1)
- net INPUT: now also RC_Connector1.3 (Pin_3)
- net VDC: now also RC_Connector1.2 (Pin_2)
Other:
- note added: "001"
- note added: "09.04.2025r"
- note added: "3x onsemi 1N4148WT schottky diodes"
- note added: "6x TOSHIBA TPN2R203NC,L1Q"
- note added: "Esc Pcb"
- note added: "Motor Feedback (BEMF)"
- note added: "Piotr Helios & Szymon Nyderek"
- note added: "Power connection"
- note removed: "LiPo 7,4V JST connector"
- moved on the sheet: J2, J3, R1, R10, R3, R4, R5, R6, R7, R8, R9, RC_Connector1
