File: photon_bldc/hardware/pcb/G071_ESC/ESC_PCB/ESC_PCB.kicad_sch (KiCad schematic)
At the start: 60 parts, among them J2 Motor_Plus, J3 Motor_Minus, Q1 NMOS, Q2 NMOS, Q3 NMOS, Q4 NMOS, Q5 NMOS, Q6 NMOS, U1 STM32G071GBUx, U2 AMS1117-5.0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

Commit message: mimi
Parts:
- removed C23, C24, C25, C26, C27, C28, C29, C30, C31, C32: 10uF, symbol Device:C
Connections:
- net VCC is gone; now on net VDC: C13.1, C14.1, C15.1, C16.1, C17.1, C18.1, C19.1, C20.1, C21.1, C22.1

Commit message: jj
Other:
- note added: "NIIGGAA"
Changed lines of the file:
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@@
+		)
+	)
+	(text "NIIGGAA\n\n"
+		(exclude_from_sim no)
+		(at 199.39 144.526 0)
+		(effects
+			(font
+				(size 12.7 12.7)
+			)
 		)
 	)

Commit message: 10.04.2025
Parts:
- removed C1: 10u, Capacitor_SMD:C_0603_1608Metric, symbol Device:C
- removed U2: AMS1117-5.0, Package_TO_SOT_SMD:SOT-223-3_TabPin2, symbol Regulator_Linear:AMS1117-5.0
- removed U3: AMS1117-3.3, Package_TO_SOT_SMD:SOT-223-3_TabPin2, symbol Regulator_Linear:AMS1117-3.3
- added TP1, TP2, TP3, TP4: TestPoint, symbol Connector:TestPoint
- added U2: ~, Package_TO_SOT_SMD:SOT-23-5, symbol ESC library:ME6119C50M5G
- added U3: ~, Package_TO_SOT_SMD:SOT-23-5, symbol ESC library:ME6119C33M5G
- C10, C11, C9: value 10uF -> 1uF
- C2, C3, C4: value 10u -> 10uF; footprint Capacitor_SMD:C_0603_1608Metric -> (none)
- C7: value 100nF -> 4.7uF
- R11: value 510 -> 1K
Connections:
- net +3.3V: now also C4.1, U3.5 (V_{OUT}); no longer C12.1, C8.1
- net +3V3: now also TP1.1; no longer C4.1, D1.2 (A), D2.2 (A), D3.2 (A), U6.4 (VCC)
- net +5V: now also C12.1, C8.1, D1.2 (A), D2.2 (A), D3.2 (A), RC_Connector1.2 (Pin_2), U6.4 (VCC), U2.5 (V_{OUT}), U3.1 (V_{IN}), U3.3 (CE); no longer C2.1
- net GND: now also TP4.1, U2.2 (V_{SS}), U3.2 (V_{SS})
- net HA: now also U1.19 (PA12/PA10); no longer U1.16 (PA8)
- net HC: now also U1.16 (PA8); no longer U1.19 (PA12/PA10)
- net LA: now also U1.15 (PB1)
- net LC: now also U1.13 (PA7); no longer U1.15 (PB1)
- net SWCLK: now also TP3.1
- net SWDIO: now also TP2.1
- net VDC: now also C2.1, U2.1 (V_{IN}), U2.3 (CE); no longer RC_Connector1.2 (Pin_2)
Other:
- note added: "3.3V"
- note added: "5V"
- note added: "PogoPads for programming"
- note removed: "NIIGGAA"
- moved on the sheet: C13, C14, C15, C16, C17, C18, C19, C20, C21, C22, J2, J3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

Commit message: jjkjk
Parts:
- added C1, C23: 10uF, symbol Device:C
- added U4: L78L06_SOT89, Package_TO_SOT_SMD:SOT-89-3, symbol Regulator_Linear:L78L06_SOT89
Connections:
- net +5V: no longer C12.1, C8.1, D1.2 (A), D2.2 (A), D3.2 (A), U6.4 (VCC)
- net GND: now also C1.2, C23.2, U4.2 (GND)
- net VDC: now also C1.1, U4.3 (IN)
- new net +6V: C12.1, C23.1, C8.1, D1.2 (A), D2.2 (A), D3.2 (A), U4.1 (OUT), U6.4 (VCC)
Other:
- note added: "5V(for BEC)"
- note added: "6V"
- note removed: "5V"

Commit message: 11.04.2025-1
Parts:
- J2: value Motor_Plus -> Plus; footprint (none) -> Connector_Wire:SolderWirePad_1x01_SMD_1x2mm
- J3: value Motor_Minus -> Minus; footprint (none) -> Connector_Wire:SolderWirePad_1x01_SMD_1x2mm
- R1, R10, R2, R3, R4, R5, R6, R7, R8, R9: footprint (none) -> Resistor_SMD:R_0603_1608Metric
Connections:
- net +5V: no longer U3.1 (V_{IN}), U3.3 (CE)
- net +6V: now also U3.1 (V_{IN}), U3.3 (CE)
Other:
- moved on the sheet: J2, J3, RC_Connector1

Commit message: sdfsdfgsdffgsdfsdsd
Parts:
- removed RC_Connector1: Conn_01x03, symbol Connector_Generic:Conn_01x03
- added TP10: PHASE_A, symbol Connector:TestPoint
- added TP5: input, TestPoint:TestPoint_Pad_2.5x2.5mm, symbol Connector:TestPoint
- added TP6: 5V, TestPoint:TestPoint_Pad_2.5x2.5mm, symbol Connector:TestPoint
- added TP7: gnd, TestPoint:TestPoint_Pad_2.5x2.5mm, symbol Connector:TestPoint
- added TP8: PHASE_C, symbol Connector:TestPoint
- added TP9: PHASE_B, symbol Connector:TestPoint
- C1, C10, C11, C12, C13, C14, C15, C16, C17, C18, C19, C2, C20, C21, C22, C23, C3, C4, C8, C9: footprint (none) -> Capacitor_SMD:C_0603_1608Metric
- TP1: value TestPoint -> 3.3V; footprint (none) -> TestPoint:TestPoint_Pad_2.0x2.0mm
- TP2: value TestPoint -> swdio; footprint (none) -> TestPoint:TestPoint_Pad_2.0x2.0mm
- TP3: value TestPoint -> swclk; footprint (none) -> TestPoint:TestPoint_Pad_2.0x2.0mm
- TP4: value TestPoint -> gnd; footprint (none) -> TestPoint:TestPoint_Pad_2.0x2.0mm
Connections:
- net +5V: now also TP6.1
- net GND: now also TP7.1
- net INPUT: now also TP5.1
- net PHASE_A: now also TP10.1
- net PHASE_B: now also TP9.1
- net PHASE_C: now also TP8.1

Commit message: 11.04.2025-2
Parts:
- removed TP8: PHASE_C, symbol Connector:TestPoint
- added TP11: T_PHASE_A, Fortior Tech FD6288Q driver library:PhasePad, symbol Connector:TestPoint
- TP10: value PHASE_A -> T_PHASE_B; footprint (none) -> Fortior Tech FD6288Q driver library:PhasePad
- TP2: value swdio -> SWDIO
- TP3: value swclk -> SWCLK
- TP4: value gnd -> GND
- TP9: value PHASE_B -> T_PHASE_C; footprint (none) -> Fortior Tech FD6288Q driver library:PhasePad
Connections:
- net PHASE_A: now also TP11.1; no longer TP10.1
- net PHASE_B: now also TP10.1; no longer TP9.1
- net PHASE_C: now also TP9.1
Other:
- moved on the sheet: TP1, TP2, TP3, TP4

Commit message: 14.04.2025r
Parts:
- TP1, TP2, TP3, TP4: footprint TestPoint:TestPoint_Pad_2.0x2.0mm -> TestPoint:TestPoint_Pad_D1.0mm
- TP5, TP6, TP7: footprint TestPoint:TestPoint_Pad_2.5x2.5mm -> Connector_Wire:SolderWirePad_1x01_SMD_1x2mm
Changed lines of the file:
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@@
 			)
 		)
-		(property "Footprint" "TestPoint:TestPoint_Pad_2.5x2.5mm"
+		(property "Footprint" "Connector_Wire:SolderWirePad_1x01_SMD_1x2mm"
 			(at 137.16 31.75 0)
 			(effects
@@
 			)
 		)
-		(property "Footprint" "TestPoint:TestPoint_Pad_2.5x2.5mm"
+		(property "Footprint" "Connector_Wire:SolderWirePad_1x01_SMD_1x2mm"
 			(at 137.16 36.83 0)
 			(effects
@@
 			)
 		)
-		(property "Footprint" "TestPoint:TestPoint_Pad_2.0x2.0mm"
+		(property "Footprint" "TestPoint:TestPoint_Pad_D1.0mm"
 			(at 245.11 137.16 0)
 			(effects
@@
 			)
 		)
-		(property "Footprint" "TestPoint:TestPoint_Pad_2.0x2.0mm"
+		(property "Footprint" "TestPoint:TestPoint_Pad_D1.0mm"
 			(at 245.11 143.51 0)
 			(effects
@@
 			)
 		)
-		(property "Footprint" "TestPoint:TestPoint_Pad_2.5x2.5mm"
+		(property "Footprint" "Connector_Wire:SolderWirePad_1x01_SMD_1x2mm"
 			(at 137.16 34.29 0)
 			(effects
@@
 			)
 		)
-		(property "Footprint" "TestPoint:TestPoint_Pad_2.0x2.0mm"
+		(property "Footprint" "TestPoint:TestPoint_Pad_D1.0mm"
 			(at 245.11 146.05 0)
 			(effects
@@
 			)
 		)
-		(property "Footprint" "TestPoint:TestPoint_Pad_2.0x2.0mm"
+		(property "Footprint" "TestPoint:TestPoint_Pad_D1.0mm"
 			(at 245.11 139.7 0)
 			(effects
