File: photon_bldc/hardware/pcb/G071_ESC/ESC_PCB/ESC_PCB.kicad_pcb (KiCad board)
At the start: 2 copper layers, 58 parts, among them J2 Plus, J3 Minus, Q1 NMOS, Q2 NMOS, Q3 NMOS, Q4 NMOS, Q5 NMOS, Q6 NMOS, U1 STM32G071GBUx, U4 L78L06_SOT89

Commit message: 11.04.2025-2
Parts:
- added TP10: T_PHASE_B, Fortior Tech FD6288Q driver library:PhasePad, F.Cu at (116.2, 59.0)
- added TP11: T_PHASE_A, Fortior Tech FD6288Q driver library:PhasePad, F.Cu at (120.2, 59.0)
- added TP9: T_PHASE_C, Fortior Tech FD6288Q driver library:PhasePad, F.Cu at (112.2, 59.0)
- TP2: value swdio -> SWDIO
- TP3: value swclk -> SWCLK
- TP4: value gnd -> GND

Commit message: gugui
Parts:
- U1, U2, U3, U4: moved to B.Cu
- moved U2 49.7 mm to (79.2, 98.6), turned to 180 degrees
- moved Q2 47.4 mm to (78.0, 91.5), turned to 90 degrees
- moved U6 45.9 mm to (82.2, 98.9)
- moved Q6 43.8 mm to (78.1, 87.1), turned to -90 degrees
- moved U3 42.6 mm to (85.3, 98.5), turned to 180 degrees
- moved Q1 42.6 mm to (86.0, 91.5), turned to 90 degrees
- moved Q3 41.9 mm to (82.0, 91.5), turned to 90 degrees
- moved TP10 41.2 mm to (82.0, 82.0)
- moved TP11 41.2 mm to (86.0, 82.0)
- moved TP9 41.2 mm to (78.0, 82.0)
- moved Q5 39.5 mm to (82.1, 87.1), turned to -90 degrees
- moved Q4 35.8 mm to (86.1, 87.1), turned to -90 degrees
- moved TP7 35.4 mm to (106.1, 102.7)
- moved U4 34.8 mm to (78.4, 85.8), turned to 180 degrees
- moved U1 24.1 mm to (82.1, 91.6), turned to 180 degrees
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Other:
- board outline added: 12 x 25 mm

Commit message: 14.04.2025r
Parts:
- C3, C4, Q1, Q2, Q3: moved to B.Cu
- J2, J3: footprint Connector_Wire:SolderWirePad_1x01_SMD_1x2mm -> Fortior Tech FD6288Q driver library:PhasePad
- TP1, TP2, TP3, TP4: footprint TestPoint:TestPoint_Pad_2.0x2.0mm -> TestPoint:TestPoint_Pad_D1.0mm
- TP5, TP6, TP7: footprint TestPoint:TestPoint_Pad_2.5x2.5mm -> Connector_Wire:SolderWirePad_1x01_SMD_1x2mm
- moved TP6 57.7 mm to (81.9, 103.6)
- moved TP5 43.0 mm to (83.5, 103.6)
- moved C1 41.2 mm to (82.7, 101.6), turned to 180 degrees
- moved C23 40.6 mm to (78.7, 98.5), turned to 180 degrees
- moved C2 37.8 mm to (82.7, 100.0), turned to 180 degrees
- moved J3 35.7 mm to (77.7, 102.1)
- moved C4 33.9 mm to (77.7, 94.5), turned to 180 degrees
- moved C3 33.0 mm to (81.0, 94.6), turned to 180 degrees
- moved TP7 25.8 mm to (80.3, 103.6)
- moved J2 25.0 mm to (86.3, 102.2)
- moved U4 17.2 mm to (82.0, 102.7), turned to -90 degrees
- moved U1 14.2 mm to (68.8, 86.5)
- moved U3 7.47 mm to (77.9, 97.5), turned to 90 degrees
- moved U6 4.40 mm to (84.5, 95.0), turned to 180 degrees
- moved Q1 4.25 mm to (86.1, 87.2)
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Routing:
- net GND: track 0.00 -> 30.0 mm, vias 0 -> 4
- net VDC: track 0.00 -> 19.1 mm, vias 0 -> 4
- net +6V: track 0.00 -> 13.2 mm, vias 0 -> 1
- net GLC: track 0.00 -> 12.6 mm, vias 0 -> 2
- net GHC: track 0.00 -> 12.1 mm, vias 0 -> 3
- net GHB: track 0.00 -> 9.58 mm, vias 0 -> 3
- net GLA: track 0.00 -> 8.26 mm, vias 0 -> 2
- net GLB: track 0.00 -> 6.72 mm, vias 0 -> 2
- net PHASE_C: track 0.00 -> 4.55 mm, vias 0 -> 3
- net PHASE_B: track 0.00 -> 4.55 mm, vias 0 -> 3
- net PHASE_A: track 0.00 -> 4.55 mm, vias 0 -> 3
- net +5V: track 0.00 -> 2.41 mm
- net +3.3V: track 0.00 -> 1.99 mm
- net GHA: track 0.00 -> 1.04 mm, vias 0 -> 1
- added copper zone on F.Cu, net GND
- added copper zone on B.Cu, net PHASE_A
- added copper zone on B.Cu, net PHASE_B
- added copper zone on B.Cu, net PHASE_C
- added copper zone on B.Cu, net VDC
Other:
- board size 12 x 25 mm -> 12 x 26 mm
- copper layers 2 -> 4

Commit message: 15.04.2025
Parts:
- removed C13, C14, C15, C16, C17, C18, C19, C20, C21, C22: 10uF, Capacitor_SMD:C_0603_1608Metric
- removed TP6: 5V, Connector_Wire:SolderWirePad_1x01_SMD_1x2mm
- added C24: 22uF, Capacitor_SMD:C_0805_2012Metric, B.Cu at (99.2, 45.8)
- added C25: 22uF, Capacitor_SMD:C_0805_2012Metric, B.Cu at (97.1, 45.8)
- added C26: 22uF, Capacitor_SMD:C_0805_2012Metric, B.Cu at (95.0, 45.8)
- added G***: LOGO, LOGO, B.Cu at (95.9, 58.5)
- C2, C5, C6, C7, R1, R10, R2, R3, R4, R5, R6, R7, R8, R9: moved to B.Cu
- C4, U3, U4: moved to F.Cu
- J2, J3: footprint Fortior Tech FD6288Q driver library:PhasePad -> Fortior Tech FD6288Q driver library:PowerPad
- moved TP7 58.3 mm to (105.1, 50.9), turned to 90 degrees
- moved J2 57.6 mm to (103.0, 47.0), turned to 90 degrees
- moved D4 56.6 mm to (91.2, 45.0)
- moved D3 56.2 mm to (84.3, 57.2), turned to 180 degrees
- moved TP5 55.2 mm to (105.1, 52.9), turned to 90 degrees
- moved U4 54.1 mm to (101.0, 52.0), turned to 0 degrees
- moved U3 54.0 mm to (97.0, 47.0), turned to 180 degrees
- moved C2 53.1 mm to (105.5, 52.0), turned to 90 degrees
- moved C1 52.2 mm to (96.5, 51.2)
- moved C23 52.2 mm to (96.5, 49.5)
- moved D2 52.1 mm to (87.5, 57.2), turned to 180 degrees
- moved J3 51.7 mm to (103.0, 57.0), turned to 90 degrees
- moved TP4 51.5 mm to (88.5, 45.0), turned to 90 degrees
- moved TP3 50.4 mm to (86.5, 45.0), turned to 90 degrees
- moved C4 50.3 mm to (94.0, 47.0), turned to 90 degrees
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Connections:
- C6 pad 1: +3V3 -> +3.3V
- C7 pad 1: +3V3 -> +3.3V
- R2 pad 1: +3V3 -> +3.3V
- TP1 pad 1: +3V3 -> +3.3V
Routing:
- net +3.3V: track 1.99 -> 46.1 mm, vias 0 -> 3
- net INPUT: track 0.00 -> 34.2 mm, vias 0 -> 2
- net GND: track 30.0 -> 54.8 mm, vias 4 -> 18
- net GHA: track 1.04 -> 23.1 mm, vias 1 -> 2
- net BEMF_REF: track 0.00 -> 22.1 mm, vias 0 -> 2
- net PHASE_C: track 4.55 -> 20.2 mm, vias 3 -> 17
- net Net-(U1-PF2): track 0.00 -> 12.8 mm
- net GHB: track 9.58 -> 22.0 mm, vias 3 -> 2
- net GHC: track 12.1 -> 23.2 mm
- net PHASE_A: track 4.55 -> 15.6 mm, vias 3 -> 17
- net SWDIO: track 0.00 -> 8.97 mm, vias 0 -> 2
- net SWCLK: track 0.00 -> 7.12 mm, vias 0 -> 2
- net BEMF_A: track 0.00 -> 6.23 mm
- net +6V: track 13.2 -> 19.3 mm, vias 1 -> 6
- net VDC: track 19.1 -> 24.8 mm, vias 4 -> 15
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- added copper zone on B.Cu, net +3.3V
- added copper zone on In1.Cu, net +5V
- added copper zone on In2.Cu, net +6V
- added copper zone on F.Cu, net PHASE_A
- added copper zone on F.Cu, net PHASE_B
- added copper zone on F.Cu, net PHASE_C
Other:
- board size 12 x 26 mm -> 36 x 16 mm
- board text added: "+5V"
- board text added: "3.3V"
- board text added: "3V3"
- board text added: "C1"
- board text added: "C10"
- board text added: "C11"
- board text added: "C12"
- board text added: "C2"
- board text added: "C23"
- board text added: "C24"
- board text added: "C25"
- board text added: "C26"
- board text added: "C3"
- board text added: "C4"
- board text added: "C5"
- board text added: "C6"
- board text added: "C7"
- board text added: "C8"
- board text added: "C9"
- board text added: "CLK"
- board text added: "D1"
- board text added: "D2"
- board text added: "D3"
- board text added: "GND"
- board text added: "PWM"
- board text added: "R1"
- board text added: "R10"
- board text added: "R11"
- board text added: "R2"
- board text added: "R3"
- board text added: "R4"
- board text added: "R5"
- board text added: "R6"
- board text added: "R7"
- board text added: "R8"
- board text added: "R9"
- board text added: "SWD"
- board text added: "VDC"

Commit message: jgguighuugi
Parts:
- added ?: , , B.Cu at (103.0, 47.0)
- added ?: , , B.Cu at (74.0, 52.0)
- added ?: , , B.Cu at (74.0, 56.0)
- added ?: , , B.Cu at (103.0, 57.0)
- added ?: , , B.Cu at (74.0, 48.0)
Routing:
- net +6V: track 19.3 -> 18.4 mm
- net GND: track 54.8 -> 54.1 mm

Commit message: 17.04.2025r-3
Parts:
- added TP6: 5V, Connector_Wire:SolderWirePad_1x01_SMD_1x2mm, F.Cu at (105.0, 51.9)
- moved TP7 0.51 mm to (105.0, 50.4)
- moved TP5 0.47 mm to (105.0, 53.3)
Routing:
- net +5V: track 1.84 -> 6.97 mm, vias 0 -> 2
Other:
- board text removed: "PWM"

Commit message: ojjojio
Parts:
- added R12: 10, Resistor_SMD:R_0603_1608Metric, F.Cu at (62.0, 40.7)
- added R13: 10, Resistor_SMD:R_0603_1608Metric, F.Cu at (62.0, 43.2)
- added R14: 10, Resistor_SMD:R_0603_1608Metric, F.Cu at (62.0, 45.8)
- added R15: 10, Resistor_SMD:R_0603_1608Metric, F.Cu at (62.0, 48.3)
- added R16: 10, Resistor_SMD:R_0603_1608Metric, F.Cu at (62.0, 50.8)
- added R17: 10, Resistor_SMD:R_0603_1608Metric, F.Cu at (62.0, 53.3)
- added R18: 100K, Resistor_SMD:R_0603_1608Metric, F.Cu at (62.0, 55.8)
- added R19: 10K, Resistor_SMD:R_0603_1608Metric, F.Cu at (62.0, 58.3)
- C6: value 4.7uF -> 100nF
- R11: footprint Capacitor_SMD:C_0603_1608Metric -> Resistor_SMD:R_0603_1608Metric
Connections:
- Q1 pad 2: GHA -> Net-(Q1-G)
- Q2 pad 2: GHC -> Net-(Q2-G)
- Q3 pad 2: GHB -> Net-(Q3-G)
- Q4 pad 2: GLA -> Net-(Q4-G)
- Q5 pad 2: GLB -> Net-(Q5-G)
- Q6 pad 2: GLC -> Net-(Q6-G)
- U1 pad 12: unconnected-(U1-PA6-Pad12) -> ADC_VOLT
