File: photon_bldc/hardware/pcb/G071_ESC/ESC_PCB/ESC_PCB.kicad_pcb (KiCad board)
At the start: 4 copper layers, 36 x 16 mm, 67 parts, among them J2 Plus, J3 Minus, Q1 NMOS, Q2 NMOS, Q3 NMOS, Q4 NMOS, Q5 NMOS, Q6 NMOS, U1 STM32G071GBUx, U4 L78L06_SOT89

Commit message: 21.03.2025r-2
Parts:
- added G***: LOGO, LOGO, F.Cu at (87.2, 45.4)
- added G***: LOGO, LOGO, F.Cu at (91.8, 51.0)
- moved C24 1.42 mm to (94.6, 47.8)
- moved C25 1.42 mm to (96.5, 47.8)
- moved C26 1.42 mm to (98.5, 47.8)
- moved TP9 0.10 mm to (74.0, 46.0)
- moved ? 0.08 mm to (104.0, 46.0)
- moved ? 0.07 mm to (104.0, 57.9)
- moved J2 0.07 mm to (104.0, 46.1)
- moved ? 0.07 mm to (74.0, 46.0)
- moved J3 0.07 mm to (104.0, 58.0)
Routing:
- net Net-(Q6-G): track 0.00 -> 1.29 mm
- net GND: track 27.9 -> 26.8 mm, vias 11 -> 26
- net PHASE_C: track 27.8 -> 27.5 mm, vias 2 -> 17
- net VDC: vias 1 -> 15
- net PHASE_B: vias 2 -> 17
- net PHASE_A: vias 2 -> 17
- net +3.3V: vias 4 -> 3
Other:
- board text added: "+5V"
- board text added: "3.3V"
- board text added: "5V"
- board text added: "6V"
- board text added: "C1"
- board text added: "C10"
- board text added: "C11"
- board text added: "C12"
- board text added: "C2"
- board text added: "C23"
- board text added: "C24"
- board text added: "C25"
- board text added: "C26"
- board text added: "C3"
- board text added: "C4"
- board text added: "C5"
- board text added: "C6"
- board text added: "C7"
- board text added: "C8"
- board text added: "C9"
- board text added: "CLK"
- board text added: "D1"
- board text added: "D2"
- board text added: "D3"
- board text added: "D4"
- board text added: "GND"
- board text added: "PWM"
- board text added: "R1"
- board text added: "R10"
- board text added: "R11"
- board text added: "R12"
- board text added: "R13"
- board text added: "R14"
- board text added: "R15"
- board text added: "R16"
- board text added: "R17"
- board text added: "R18"
- board text added: "R19"
- board text added: "R2"
- board text added: "R3"
- board text added: "R4"
- board text added: "R5"
- board text added: "R6"
- board text added: "R7"
- board text added: "R8"
- board text added: "R9"
- board text added: "SWD"
- board text added: "VDC"

Commit message: 21.04.2025
Routing:
- net VDC: vias 15 -> 25

Commit message: 22.04.2025
Parts:
- C1, C2, C23, C3, C4, C8: footprint Capacitor_SMD:C_0402_1005Metric_Pad0.74x0.62mm_HandSolder -> Capacitor_SMD:C_0603_1608Metric_Pad1.08x0.95mm_HandSolder
- moved C1 6.00 mm to (97.3, 50.3), turned to -90 degrees
- moved C3 0.94 mm to (94.1, 47.0)
- moved U2 0.79 mm to (97.0, 46.9)
- moved C8 0.67 mm to (83.2, 48.8)
- moved C12 0.48 mm to (83.7, 47.5)
- moved D4 0.44 mm to (94.6, 55.6)
- moved C2 0.43 mm to (100.2, 47.2), turned to -90 degrees
- moved R11 0.38 mm to (97.0, 53.3)
- moved C23 0.29 mm to (99.2, 58.5)
Routing:
- net VDC: track 12.0 -> 17.2 mm
- net +5V: track 15.9 -> 17.5 mm
- net GND: track 26.8 -> 28.4 mm
- net Net-(D4-K): track 2.16 -> 2.87 mm
