File: photon_bldc/hardware/pcb/G071_ESC/ESC_PCB/ESC_PCB.kicad_pcb (KiCad board)
At the start: 4 copper layers, 36 x 16 mm, 69 parts, among them J2 Plus, J3 Minus, Q1 NMOS, Q2 NMOS, Q3 NMOS, Q4 NMOS, Q5 NMOS, Q6 NMOS, U1 STM32G071GBUx, U4 L78L06_SOT89

Commit message: 11.05.2025r
Changed lines of the file:
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@@
 	)
 	(segment
-		(start 87.2 53.9)
-		(end 87.03 53.9)
+		(start 87.2 53.55)
+		(end 87.15 53.5)
 		(width 0.15)
 		(layer "F.Cu")
@@
 	)
 	(segment
-		(start 87.03 53.9)
+		(start 87.2 53.9)
+		(end 87.2 53.55)
+		(width 0.15)
+		(layer "F.Cu")
+		(net 14)
+	)
+	(segment
+		(start 87.15 53.5)
 		(end 86.63 53.5)
 		(width 0.15)

Commit message: esc
Parts:
- removed ? (x5): , 
- removed C5: 100nF, Capacitor_SMD:C_0402_1005Metric_Pad0.74x0.62mm_HandSolder
- removed G*** (x2): LOGO, LOGO
- removed R2: 10k, Resistor_SMD:R_0402_1005Metric_Pad0.72x0.64mm_HandSolder
- C1, C2, C3, C4: footprint Capacitor_SMD:C_0603_1608Metric_Pad1.08x0.95mm_HandSolder -> Capacitor_SMD:C_0402_1005Metric_Pad0.74x0.62mm_HandSolder
- C10, C11, C8, C9, D1, D2, D3, U6: moved to B.Cu
- C12: footprint Capacitor_SMD:C_0402_1005Metric_Pad0.74x0.62mm_HandSolder -> Capacitor_SMD:C_0201_0603Metric_Pad0.64x0.40mm_HandSolder; moved to B.Cu
- C24, C25, C26: moved to F.Cu
- C6: footprint Capacitor_SMD:C_0402_1005Metric_Pad0.74x0.62mm_HandSolder -> Capacitor_SMD:C_0201_0603Metric_Pad0.64x0.40mm_HandSolder
- D4: footprint LED_SMD:LED_0603_1608Metric -> LED_SMD:LED_0201_0603Metric_Pad0.64x0.40mm_HandSolder
- Q1, Q2, Q3: footprint Fortior Tech FD6288Q driver library:TSON-8(3.1x3.1) -> MOSFET_lib:NCEP3065
- Q4, Q5, Q6: footprint Fortior Tech FD6288Q driver library:TSON-8(3.1x3.1) -> MOSFET_lib:NCEP3065; moved to B.Cu
- R1, R10, R11, R12, R13, R14, R15, R16, R17, R18, R19, R3, R4, R5, R6, R7, R8, R9: footprint Resistor_SMD:R_0402_1005Metric_Pad0.72x0.64mm_HandSolder -> Resistor_SMD:R_0201_0603Metric_Pad0.64x0.40mm_HandSolder
- moved R14 93.7 mm to (150.3, 107.8), turned to 0 degrees
- moved R12 91.1 mm to (150.2, 109.5), turned to 0 degrees
- moved R16 91.0 mm to (150.2, 110.4), turned to 0 degrees
- moved R18 90.9 mm to (140.9, 118.3), turned to 90 degrees
- moved R19 90.0 mm to (141.9, 118.3), turned to -90 degrees
- moved C26 86.0 mm to (149.9, 116.8), turned to 0 degrees
- moved TP4 85.9 mm to (150.9, 121.0), turned to 180 degrees
- moved C25 85.6 mm to (149.9, 114.8), turned to 0 degrees
- moved C24 85.3 mm to (149.9, 112.7), turned to 0 degrees
- moved R4 84.9 mm to (144.0, 119.2), turned to 180 degrees
- moved Q6 84.0 mm to (142.2, 100.8)
- moved C12 84.0 mm to (142.3, 107.7), turned to 90 degrees
- moved TP11 83.8 mm to (150.8, 91.3)
- moved R6 83.6 mm to (141.4, 115.0)
- moved R15 83.6 mm to (141.2, 103.5)
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Connections:
- U1 pad 5: Net-(U1-PF2) -> unconnected-(U1-PF2-Pad5)
Routing:
- net GND: track 28.4 -> 0.00 mm, vias 26 -> 0
- net INPUT: track 28.2 -> 0.00 mm, vias 2 -> 0
- net PHASE_C: track 27.5 -> 0.00 mm, vias 17 -> 0
- net +6V: track 23.9 -> 0.00 mm, vias 4 -> 0
- net PHASE_B: track 20.4 -> 0.00 mm, vias 17 -> 0
- net +5V: track 17.5 -> 0.00 mm, vias 2 -> 0
- net VDC: track 17.2 -> 0.00 mm, vias 25 -> 0
- net SWDIO: track 14.6 -> 0.00 mm, vias 2 -> 0
- net +3.3V: track 13.9 -> 0.00 mm, vias 3 -> 0
- net PHASE_A: track 11.5 -> 0.00 mm, vias 17 -> 0
- net SWCLK: track 11.3 -> 0.00 mm, vias 2 -> 0
- net BEMF_REF: track 11.2 -> 0.00 mm, vias 2 -> 0
- net GHA: track 11.1 -> 0.00 mm, vias 2 -> 0
- net GHC: track 11.0 -> 0.00 mm, vias 2 -> 0
- net GHB: track 8.37 -> 0.00 mm, vias 2 -> 0
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- removed copper zone on B.Cu, net +3.3V
- removed copper zone on In2.Cu, net +6V
- removed copper zone on F.Cu, net GND
- removed copper zone on In1.Cu, net GND
- removed copper zone on B.Cu, net PHASE_A
- removed copper zone on F.Cu, net PHASE_A
- removed copper zone on B.Cu, net PHASE_B
- removed copper zone on F.Cu, net PHASE_B
- removed copper zone on B.Cu, net PHASE_C
- removed copper zone on F.Cu, net PHASE_C
- removed copper zone on B.Cu, net VDC
- removed copper zone on In1.Cu, net VDC
Other:
- board size 36 x 16 mm -> 12 x 32 mm
- board text removed: "+5V"
- board text removed: "3.3V"
- board text removed: "5V"
- board text removed: "6V"
- board text removed: "C1"
- board text removed: "C10"
- board text removed: "C11"
- board text removed: "C12"
- board text removed: "C2"
- board text removed: "C23"
- board text removed: "C24"
- board text removed: "C25"
- board text removed: "C26"
- board text removed: "C3"
- board text removed: "C4"
- board text removed: "C5"
- board text removed: "C6"
- board text removed: "C7"
- board text removed: "C8"
- board text removed: "C9"
- board text removed: "CLK"
- board text removed: "D1"
- board text removed: "D2"
- board text removed: "D3"
- board text removed: "D4"
- board text removed: "GND"
- board text removed: "PWM"
- board text removed: "R1"
- board text removed: "R10"
- board text removed: "R11"
- board text removed: "R12"
- board text removed: "R13"
- board text removed: "R14"
- board text removed: "R15"
- board text removed: "R16"
- board text removed: "R17"
- board text removed: "R18"
- board text removed: "R19"
- board text removed: "R2"
- board text removed: "R3"
- board text removed: "R4"
- board text removed: "R5"
- board text removed: "R6"
- board text removed: "R7"
- board text removed: "R8"
- board text removed: "R9"
- board text removed: "SWD"
- board text removed: "VDC"

Commit message: oefvoj
Parts:
- C1, C2, C23, C24, C25, C26, C3, C4, D4, R11, U2, U3, U4: moved to B.Cu
- C10, C11, C12, C6, C7, C8, C9, D1, D2, D3, R1, R10, R12, R14, R16, R3, R4, R5, R6, R7, R8, R9, TP1, TP2, TP3, TP4, U1, U6: moved to F.Cu
- moved TP4 15.1 mm to (141.0, 109.6), turned to 0 degrees
- moved TP3 15.1 mm to (141.0, 108.0), turned to 0 degrees
- moved TP1 15.0 mm to (141.1, 104.8), turned to 0 degrees
- moved TP2 15.0 mm to (141.1, 106.3), turned to 0 degrees
- moved R14 13.6 mm to (144.6, 95.5)
- moved U4 12.8 mm to (147.0, 119.4), turned to 0 degrees
- moved C1 12.7 mm to (143.6, 117.5), turned to -90 degrees
- moved C23 12.2 mm to (143.4, 120.3)
- moved R12 11.9 mm to (144.6, 99.0)
- moved R15 11.6 mm to (149.6, 95.5), turned to 0 degrees
- moved C8 10.5 mm to (151.2, 107.3)
- moved Q6 9.84 mm to (149.7, 94.5), turned to 90 degrees
- moved R7 9.78 mm to (150.8, 115.7)
- moved Q1 9.75 mm to (144.7, 101.5), turned to 90 degrees
- moved R16 9.70 mm to (144.6, 102.5)
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Routing:
- net Net-(Q6-G): vias 0 -> 1
- net Net-(Q5-G): vias 0 -> 1
- net Net-(Q4-G): vias 0 -> 1
- net Net-(Q3-G): vias 0 -> 1
- net Net-(Q2-G): vias 0 -> 1
- net Net-(Q1-G): vias 0 -> 1

Commit message: wdads
Parts:
- added ?: , , B.Cu at (146.2, 91.2)
- added ?: , , B.Cu at (150.8, 120.3)
- added ?: , , B.Cu at (142.4, 91.2)
- added ?: , , B.Cu at (149.8, 91.2)
- added ?: , , B.Cu at (141.2, 120.3)
- moved R19 11.6 mm to (143.5, 108.5), turned to 90 degrees
- moved R18 11.4 mm to (142.3, 109.0), turned to 0 degrees
- moved TP11 7.15 mm to (142.4, 91.3)
- moved TP10 3.80 mm to (149.8, 91.3)
- moved TP9 3.55 mm to (146.1, 91.3)
- moved Q2 0.42 mm to (144.7, 94.9)
- moved Q6 0.42 mm to (149.7, 94.9)
- moved R15 0.40 mm to (149.6, 95.9)
- moved R14 0.40 mm to (144.6, 95.9)
- moved Q3 0.20 mm to (144.7, 98.2)
- moved Q5 0.20 mm to (149.7, 98.2)
- moved R13 0.20 mm to (149.6, 99.2)
- moved R12 0.18 mm to (144.6, 99.2)
- moved R17 0.06 mm to (149.6, 102.5)
Routing:
- added copper zone on B.Cu, net GND
- added copper zone on B.Cu, net PHASE_A
- added copper zone on F.Cu, net PHASE_A
- added copper zone on B.Cu, net PHASE_B
- added copper zone on F.Cu, net PHASE_B
- added copper zone on In1.Cu, net PHASE_B
- added copper zone on In2.Cu, net PHASE_B
- added copper zone on In3.Cu, net PHASE_B
- added copper zone on In4.Cu, net PHASE_B
- added copper zone on B.Cu, net PHASE_C
- added copper zone on F.Cu, net PHASE_C
- added copper zone on In1.Cu, net PHASE_C
- added copper zone on In2.Cu, net PHASE_C
- added copper zone on In3.Cu, net PHASE_C
- added copper zone on In4.Cu, net PHASE_C
- added copper zone on B.Cu, net VDC
- added copper zone on In1.Cu, net VDC
- added copper zone on In2.Cu, net VDC
- added copper zone on In3.Cu, net VDC
- added copper zone on In4.Cu, net VDC
Other:
- copper layers 4 -> 6

Commit message: dvbdfbdfb
Parts:
- R10, R5, R6, R7, R8, R9: moved to B.Cu
- moved R5 11.2 mm to (148.9, 103.7)
- moved R7 10.6 mm to (148.9, 105.3)
- moved R9 10.2 mm to (148.8, 108.8), turned to 180 degrees
- moved R10 10.2 mm to (148.8, 107.8), turned to 180 degrees
- moved R8 10.1 mm to (148.8, 106.8), turned to 0 degrees
- moved R6 9.39 mm to (148.9, 104.5)
- moved R1 8.41 mm to (142.4, 111.2)
- moved R3 8.41 mm to (142.4, 112.2)
- moved R4 8.41 mm to (142.4, 113.2)
Routing:
- net VDC: track 0.00 -> 11.8 mm, vias 0 -> 1
- net +6V: track 0.00 -> 5.22 mm, vias 0 -> 2
- net +3.3V: track 0.00 -> 3.53 mm, vias 0 -> 2
- net +5V: track 0.00 -> 1.94 mm, vias 0 -> 1
- net Net-(D4-K): track 0.00 -> 0.94 mm
- net PHASE_C: vias 0 -> 1
- net PHASE_B: vias 0 -> 1
- net PHASE_A: vias 0 -> 1
- net GND: vias 0 -> 2
- added copper zone on In2.Cu, net +5V
- added copper zone on F.Cu, net GND
- added copper zone on In1.Cu, net GND
- added copper zone on In2.Cu, net GND
- added copper zone on In3.Cu, net GND
- added copper zone on In4.Cu, net GND
- added copper zone on In1.Cu, net PHASE_A
- added copper zone on In2.Cu, net PHASE_A
- added copper zone on In3.Cu, net PHASE_A
- added copper zone on In4.Cu, net PHASE_A

Commit message: ghjhbk
Parts:
- turned C11 to 90 degrees
- turned D3 to 90 degrees
Routing:
- net PHASE_C: track 0.00 -> 25.0 mm, vias 1 -> 7
- net BEMF_REF: track 0.00 -> 19.1 mm, vias 0 -> 1
- net BEMF_A: track 0.00 -> 16.3 mm
- net PHASE_A: track 0.00 -> 16.0 mm, vias 1 -> 7
- net PHASE_B: track 0.00 -> 13.1 mm, vias 1 -> 8
- net SWDIO: track 0.00 -> 8.98 mm
- net Net-(D1-K): track 0.00 -> 8.24 mm, vias 0 -> 1
- net SWCLK: track 0.00 -> 7.05 mm
- net Net-(D3-K): track 0.00 -> 5.61 mm
- net Net-(U6-VS3): track 0.00 -> 3.30 mm
- net +3.3V: track 3.53 -> 6.30 mm, vias 2 -> 3
- net GND: track 0.00 -> 2.65 mm, vias 2 -> 4
- net BEMF_C: track 0.00 -> 2.07 mm
- net BEMF_B: track 0.00 -> 1.60 mm
- net +5V: vias 1 -> 2
- added copper zone on In3.Cu, net +3.3V

Commit message: dfbdfb
Parts:
- moved R19 1.16 mm to (142.7, 107.7)
Routing:
- net +6V: track 5.22 -> 16.8 mm, vias 2 -> 4
- net Net-(U6-VS1): track 0.00 -> 11.5 mm, vias 0 -> 2
- net Net-(D2-K): track 0.00 -> 10.0 mm, vias 0 -> 2
- net Net-(U6-VS2): track 0.00 -> 9.14 mm, vias 0 -> 2
- net BEMF_C: track 2.07 -> 10.9 mm, vias 0 -> 2
- net INPUT: track 0.00 -> 8.55 mm
- net GND: track 2.65 -> 4.22 mm
- net Net-(D1-K): track 8.24 -> 9.58 mm
- net ADC_VOLT: track 0.00 -> 0.89 mm

Commit message: dvf
Routing:
- net GHA: track 0.00 -> 11.2 mm
- net GLA: track 0.00 -> 7.41 mm
- net Net-(U6-VS1): track 11.5 -> 10.8 mm
- net SWCLK: track 7.05 -> 6.36 mm
- net SWDIO: track 8.98 -> 8.30 mm
- net PHASE_A: track 16.0 -> 15.7 mm, vias 7 -> 6
