File: photon_bldc/hardware/pcb/G071_ESC/ESC_PCB/_autosave-ESC_PCB.kicad_pcb (KiCad board)
At the start: 4 copper layers, 36 x 16 mm, 67 parts, among them J2 Plus, J3 Minus, Q1 NMOS, Q2 NMOS, Q3 NMOS, Q4 NMOS, Q5 NMOS, Q6 NMOS, U1 STM32G071GBUx, U4 L78L06_SOT89

Commit message: 21.04.2025
Parts:
- added G***: LOGO, LOGO, F.Cu at (87.2, 45.4)
- added G***: LOGO, LOGO, F.Cu at (91.8, 51.0)
- moved C24 1.42 mm to (94.6, 47.8)
- moved C25 1.42 mm to (96.5, 47.8)
- moved C26 1.42 mm to (98.5, 47.8)
- moved TP9 0.10 mm to (74.0, 46.0)
- moved ? 0.08 mm to (104.0, 46.0)
- moved ? 0.07 mm to (104.0, 57.9)
- moved J2 0.07 mm to (104.0, 46.1)
- moved ? 0.07 mm to (74.0, 46.0)
- moved J3 0.07 mm to (104.0, 58.0)
Routing:
- net PHASE_C: track 27.8 -> 11.7 mm, vias 2 -> 17
- net Net-(Q6-G): track 0.00 -> 1.29 mm
- net GND: track 27.9 -> 26.8 mm, vias 11 -> 26
- net VDC: vias 1 -> 15
- net PHASE_B: vias 2 -> 17
- net PHASE_A: vias 2 -> 17
Other:
- board text added: "+5V"
- board text added: "3.3V"
- board text added: "5V"
- board text added: "6V"
- board text added: "C1"
- board text added: "C10"
- board text added: "C11"
- board text added: "C12"
- board text added: "C2"
- board text added: "C23"
- board text added: "C24"
- board text added: "C25"
- board text added: "C26"
- board text added: "C3"
- board text added: "C4"
- board text added: "C5"
- board text added: "C6"
- board text added: "C7"
- board text added: "C8"
- board text added: "C9"
- board text added: "CLK"
- board text added: "D1"
- board text added: "D2"
- board text added: "D3"
- board text added: "D4"
- board text added: "GND"
- board text added: "PWM"
- board text added: "R1"
- board text added: "R10"
- board text added: "R11"
- board text added: "R12"
- board text added: "R13"
- board text added: "R14"
- board text added: "R15"
- board text added: "R16"
- board text added: "R17"
- board text added: "R18"
- board text added: "R19"
- board text added: "R2"
- board text added: "R3"
- board text added: "R4"
- board text added: "R5"
- board text added: "R6"
- board text added: "R7"
- board text added: "R8"
- board text added: "R9"
- board text added: "SWD"
- board text added: "VDC"
