File: photon_bldc/hardware/pcb/Main_board/main_board/main_board.kicad_sch (KiCad schematic)
At the start: 51 parts, among them J1 -VIN+, J2 Micro_SD_Card, J3 Conn_01x18, SW1 SW_DPDT_x2, SW2 SW_SPST, U1 STM32G474RETx, U2 AMS1117-5.0, U3 AMS1117-3.3, U5 SST25VF080B-50-4x-S2Ax, X1 24Mhz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

Commit message: jknj
Parts:
- added Turbo1: Conn_01x02, APhotonLibrary:PowerConn, symbol Connector_Generic:Conn_01x02
Connections:
- net GND: now also Turbo1.1 (Pin_1)
- net VDC: now also Turbo1.2 (Pin_2)
Changed lines of the file:
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@@
 	(label "HSE_OUT"
 		(at 88.9 73.66 0)
+		(fields_autoplaced yes)
 		(effects
 			(font
@@
 	(label "LSE_IN"
 		(at 86.868 119.38 0)
+		(fields_autoplaced yes)
 		(effects
 			(font
@@
 	(label "LSE_OUT"
 		(at 86.868 121.92 0)
+		(fields_autoplaced yes)
 		(effects
 			(font
@@
 	(label "HSE_IN"
 		(at 88.9 71.12 0)
+		(fields_autoplaced yes)
 		(effects
 			(font
@@
 	)
 	(symbol
+		(lib_id "power:VDC")
+		(at 304.8 229.87 270)
+		(unit 1)
+		(exclude_from_sim no)
+		(in_bom yes)
+		(on_board yes)
+		(dnp no)
+		(property "Reference" "#PWR066"
+			(at 302.26 229.87 0)
+			(effects
+				(font
+					(size 1.27 1.27)
+				)
+				(hide yes)
+			)
+		)
+		(property "Value" "VDC"
+			(at 309.626 229.87 90)
+			(effects
+				(font
+					(size 1.27 1.27)
+				)
+			)
+		)
+		(property "Footprint" ""
+			(at 304.8 229.87 0)
+			(effects
+				(font
+					(size 1.27 1.27)
+				)
+				(hide yes)
+			)
+		)
+		(property "Datasheet" ""
+			(at 304.8 229.87 0)
+			(effects
+				(font
+					(size 1.27 1.27)
+				)
+				(hide yes)
+			)
+		)
+		(property "Description" ""
+			(at 304.8 229.87 0)
+			(effects
+				(font
+					(size 1.27 1.27)
+				)
+				(hide yes)
+			)
+		)
+		(pin "1"
+		)
+		(instances
+			(project "main_board"
+				(path "/1e458b73-232f-493d-9935-9a4b4c039b92"
+					(reference "#PWR066")
+					(unit 1)
+				)
+			)
+		)
+	)
+	(symbol
 		(lib_id "power:+5V")
 		(at 295.91 68.58 90)
@@
 	)
 	(symbol
+		(lib_id "Connector_Generic:Conn_01x02")
+		(at 299.72 232.41 180)
+		(unit 1)
+		(exclude_from_sim no)
+		(in_bom yes)
+		(on_board yes)
+		(dnp no)
+		(property "Reference" "Turbo1"
+			(at 318.008 231.14 0)
+			(effects
+				(font
+					(size 1.27 1.27)
+				)
+			)
+		)
+		(property "Value" "Conn_01x02"
+			(at 299.72 226.06 0)
+			(effects
+				(font
+					(size 1.27 1.27)
+				)
+				(hide yes)
+			)
+		)
+		(property "Footprint" "APhotonLibrary:PowerConn"
+			(at 299.72 232.41 0)
+			(effects
+				(font
+					(size 1.27 1.27)
+				)
+				(hide yes)
+			)
+		)
+		(property "Datasheet" "~"
+			(at 299.72 232.41 0)
+			(effects
+				(font
+					(size 1.27 1.27)
+				)
+				(hide yes)
+			)
+		)
+		(property "Description" "Generic connector, single row, 01x02, script generated (kicad-library-utils/schlib/autogen/connector/)"
+			(at 299.72 232.41 0)
+			(effects
+				(font
+					(size 1.27 1.27)
+				)
+				(hide yes)
+			)
+		)
+		(pin "2"
+		)
+		(pin "1"
+		)
+		(instances
+			(project "main_board"
+				(path "/1e458b73-232f-493d-9935-9a4b4c039b92"
+					(reference "Turbo1")
+					(unit 1)
+				)
+			)
+		)
+	)
+	(symbol
 		(lib_id "Device:C")
 		(at 90.424 43.688 0)
@@
 					(unit 1)
 				)
+			)
+		)
+	)
+	(symbol
+		(lib_id "power:GND")
+		(at 304.8 232.41 90)
+		(unit 1)
+		(exclude_from_sim no)
+		(in_bom yes)
+		(on_board yes)
+		(dnp no)
+		(property "Reference" "#PWR067"
+			(at 311.15 232.41 0)
+			(effects
+				(font
+					(size 1.27 1.27)
+				)
+				(hide yes)
+			)
+		)
+		(property "Value" "GND"
+			(at 309.372 232.41 90)
+			(effects
+				(font
+					(size 1.27 1.27)
+				)
+			)
+		)
+		(property "Footprint" ""
+			(at 304.8 232.41 0)
+			(effects
+				(font
+					(size 1.27 1.27)
+				)
+				(hide yes)
+			)
+		)
+		(property "Datasheet" ""
+			(at 304.8 232.41 0)
+			(effects
+				(font
+					(size 1.27 1.27)
+				)
+				(hide yes)
+			)
+		)
+		(property "Description" ""
+			(at 304.8 232.41 0)
+			(effects
+				(font
+					(size 1.27 1.27)
+				)
+				(hide yes)
+			)
+		)
+		(pin "1"
+		)
+		(instances
+			(project "main_board"
+				(path "/1e458b73-232f-493d-9935-9a4b4c039b92"
+					(reference "#PWR067")
+					(unit 1)
+				)

Commit message: 07.05.2025r-MainPCB
sd
Parts:
- added U6: ~, APhotonLibrary:ICM_MOUNT, symbol PhotonLib:ICM_MOUNT
Connections:
- net +3.3V: now also U6.5 (Vcc)
- net GND: now also U6.6 (GND)
- net SPI3_CS: now also U6.4 (CS)
- net SPI3_INT: now also U6.7 (INT)
- net SPI3_MISO: now also U6.1 (MISO)
- net SPI3_MOSI: now also U6.2 (MOSI)
- net SPI3_SCL: now also U6.3 (SCK)
Other:
- note added: "IMU -> ICM4688p"
- note added: "IMU allows the robot to know it's rotation on the track"
- moved on the sheet: Encoder_L1, Encoder_R1, MotorsPower1, MotorsPower2, PWML1, PWMR1, PWMT1, Turbo1
