File: photon_bldc/hardware/pcb/Main_board/main_board/main_board.kicad_pcb (KiCad board)
At the start: 4 copper layers, 100 x 64 mm, 55 parts, among them J1 -VIN+, J2 Micro_SD_Card, J3 Conn_01x18, SW1 SW_DPDT_x2, SW2 SW_SPST, U1 STM32G474RETx, U2 AMS1117-5.0, U3 AMS1117-3.3, U5 SST25VF080B-50-4x-S2Ax, X1 24Mhz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

Commit message: jknj
Parts:
- added Turbo1: Conn_01x02, APhotonLibrary:PowerConn, B.Cu at (182.0, 81.2)
- MotorsPower1, MotorsPower2: moved to B.Cu
- moved MotorsPower1 122.2 mm to (88.0, 97.6), turned to 90 degrees
- moved J1 30.5 mm to (170.3, 106.8), turned to 180 degrees
- moved MotorsPower2 29.4 mm to (182.0, 97.2), turned to 90 degrees
- moved PWMT1 26.1 mm to (181.7, 81.7), turned to 90 degrees
- moved C13 21.7 mm to (172.4, 77.1)
- moved C14 21.7 mm to (169.1, 77.0)
- moved C15 21.7 mm to (165.6, 77.2)
- moved C16 21.7 mm to (161.4, 77.2)
- moved R5 21.7 mm to (174.8, 75.7)
- moved R6 21.7 mm to (174.8, 72.7)
- moved U3 21.7 mm to (162.3, 82.5)
- moved U2 21.7 mm to (170.2, 82.3)
Routing:
- net VDC: track 30.5 -> 244.1 mm, vias 0 -> 15
- net GND: track 79.4 -> 94.8 mm, vias 34 -> 46
- net PWM_T: track 93.2 -> 98.0 mm

Commit message: 07.05.2025r-MainPCB
sd
Parts:
- added U6: ~, APhotonLibrary:ICM_MOUNT, F.Cu at (103.2, 84.9)
Routing:
- net LED_3: track 1.22 -> 104.2 mm, vias 1 -> 3
- net LED_4: track 1.38 -> 96.5 mm, vias 1 -> 3
- net +5V: track 20.0 -> 65.4 mm, vias 4 -> 5
- net PWM_T: track 98.0 -> 122.3 mm, vias 1 -> 3
- net SPI3_INT: track 2.03 -> 23.0 mm
- net ADC1_IN15_Batt: track 80.0 -> 100.5 mm
- net GND: track 94.8 -> 111.2 mm, vias 46 -> 49
- net SPI3_MISO: track 1.53 -> 15.1 mm
- net SPI3_MOSI: track 1.83 -> 14.2 mm
- net SPI3_SCL: track 2.23 -> 11.6 mm
- net VDC: track 244.1 -> 249.1 mm
- net SPI3_CS: track 1.88 -> 6.67 mm
- net +3.3V: track 17.1 -> 19.6 mm, vias 6 -> 7
- net Net-(D3-A): track 0.00 -> 1.82 mm
- net Net-(D4-A): track 0.00 -> 1.71 mm
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
Commit message: gjvgj
Parts:
- moved C9 1.13 mm to (94.2, 77.4)
- moved R2 0.16 mm to (107.4, 60.6)
- moved R1 0.15 mm to (103.2, 63.7)
- moved D2 0.10 mm to (108.3, 61.8)
- moved D1 0.07 mm to (104.2, 65.0)
- moved J3 0.05 mm to (135.0, 48.7)
Routing:
- net GND: track 111.2 -> 120.3 mm, vias 49 -> 55
- net UART1_RX: track 85.2 -> 82.2 mm
- net VDC: track 249.1 -> 251.0 mm
- net UART1_TX: track 81.7 -> 80.0 mm
- net LED_1: track 28.8 -> 27.4 mm
- net LED_2: track 34.4 -> 33.0 mm
- net +3.3V: track 19.6 -> 20.4 mm
- net Sensor8: vias 0 -> 1
- net (no net): vias 1 -> 0
