File: photon_bldc/hardware/pcb/one_sided_main_board/main_board.kicad_pcb (KiCad board)
At the start: 4 copper layers, 100 x 64 mm, 48 parts, among them J1 -VIN+, J2 Micro_SD_Card, J3 Conn_01x18, SW2 SW_SPST, U1 STM32G474RETx, U2 AMS1117-5.0, U3 AMS1117-3.3, U5 SST25VF080B-50-4x-S2Ax, X1 24Mhz, X2 32.768KHz

Commit message: dfhdfh
Other:
- board text added: "9.05.2025"
- board text added: "Piotr Helios Szymon Nyderek"
Changed lines of the file:
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@@
 		(tags "resistor")
 		(property "Reference" "R2"
-			(at -2.475 -0.15 360)
+			(at -2.475 -0.15 0)
 			(layer "F.SilkS")
 			(effects
@@
 		)
 		(property "Value" "510R"
-			(at 0 1.43 360)
+			(at 0 1.43 0)
 			(layer "F.Fab")
 			(effects
@@
 		)
 		(fp_text user "${REFERENCE}"
-			(at 0 0 360)
+			(at 0 0 0)
 			(layer "F.Fab")
 			(effects
@@
 		(tags "resistor")
 		(property "Reference" "R1"
-			(at -0.05 1.4 360)
+			(at -0.05 1.4 0)
 			(layer "F.SilkS")
 			(effects
@@
 		)
 		(property "Value" "510R"
-			(at 0 1.43 360)
+			(at 0 1.43 0)
 			(layer "F.Fab")
 			(effects
@@
 		)
 		(fp_text user "${REFERENCE}"
-			(at 0 0 360)
+			(at 0 0 0)
 			(layer "F.Fab")
 			(effects
@@
 		(layer "Edge.Cuts")
 	)
+	(gr_text "9.05.2025"
+		(at 86.075 108.4 -90)
+		(layer "B.SilkS")
+		(effects
+			(font
+				(size 1 1)
+				(thickness 0.15)
+			)
+			(justify left bottom mirror)
+		)
+	)
+	(gr_text "Piotr Helios \nSzymon Nyderek"
+		(at 86.05 85.575 270)
+		(layer "B.SilkS")
+		(effects
+			(font
+				(size 1 1)
+				(thickness 0.15)
+			)
+			(justify bottom mirror)
+		)
+	)
 	(gr_text "HC-04"
 		(at 162.25 76.85 0)
@@
 	)
 	(segment
-		(start 111.9 78.9)
-		(end 111.65 79.15)
-		(width 0.15)
-		(layer "In1.Cu")
-		(net 34)
-	)
-	(segment
-		(start 111.65 87.1)
+		(start 111.9 87.35)
 		(end 127.05 102.5)
 		(width 0.15)
@@
 	)
 	(segment
-		(start 111.65 79.15)
-		(end 111.65 87.1)
+		(start 111.9 78.9)
+		(end 111.9 87.35)
 		(width 0.15)
 		(layer "In1.Cu")
@@
 	)
 	(segment
-		(start 113.05 86.3)
-		(end 128.2 101.45)
+		(start 151.65 101.25)
+		(end 157.2 95.7)
 		(width 0.15)
 		(layer "In1.Cu")
@@
 	)
 	(segment
-		(start 128.2 101.45)
-		(end 151.7 101.45)
+		(start 113.05 86.3)
+		(end 128 101.25)
 		(width 0.15)
 		(layer "In1.Cu")
@@
 	)
 	(segment
-		(start 112.465331 77.4)
-		(end 112.465331 77.842892)
+		(start 113.05 78.427561)
+		(end 113.05 86.3)
 		(width 0.15)
 		(layer "In1.Cu")
@@
 	)
 	(segment
-		(start 151.7 101.45)
-		(end 157.2 95.95)
+		(start 128 101.25)
+		(end 151.65 101.25)
 		(width 0.15)
 		(layer "In1.Cu")
@@
 	)
 	(segment
-		(start 157.2 95.95)
+		(start 157.2 95.7)
 		(end 157.2 93.2)
 		(width 0.15)
@@
 	)
 	(segment
-		(start 113.05 78.427561)
-		(end 113.05 86.3)
+		(start 112.465331 77.842892)
+		(end 113.05 78.427561)
 		(width 0.15)
 		(layer "In1.Cu")
@@
 	)
 	(segment
-		(start 112.465331 77.842892)
-		(end 113.05 78.427561)
+		(start 112.465331 77.4)
+		(end 112.465331 77.842892)
 		(width 0.15)
 		(layer "In1.Cu")
@@
 	)
 	(segment
-		(start 112.315332 78.4)
-		(end 112.55 78.634668)
+		(start 112.45 78.534668)
+		(end 112.45 86.8)
 		(width 0.15)
 		(layer "In1.Cu")
@@
 	)
 	(segment
-		(start 157.75 96.05)
-		(end 157.75 91.4)
+		(start 151.95 101.85)
+		(end 157.75 96.05)
 		(width 0.15)
 		(layer "In1.Cu")
@@
 	)
 	(segment
-		(start 151.95 101.85)
-		(end 157.75 96.05)
+		(start 157.75 91.4)
+		(end 157.35 91)
 		(width 0.15)
 		(layer "In1.Cu")
@@
 	)
 	(segment
-		(start 112.55 78.634668)
-		(end 112.55 86.9)
+		(start 112.315332 78.4)
+		(end 112.45 78.534668)
 		(width 0.15)
 		(layer "In1.Cu")
@@
 	)
 	(segment
-		(start 157.75 91.4)
-		(end 157.35 91)
+		(start 112.45 86.8)
+		(end 127.5 101.85)
 		(width 0.15)
 		(layer "In1.Cu")
@@
 	)
 	(segment
-		(start 112.55 86.9)
-		(end 127.5 101.85)
+		(start 157.75 96.05)
+		(end 157.75 91.4)
 		(width 0.15)
 		(layer "In1.Cu")
@@
 	)
 	(segment
-		(start 91.6 82.3)
-		(end 91.6 80.05)
-		(width 0.15)
-		(layer "In1.Cu")
-		(net 42)
-	)
-	(segment
-		(start 102.492893 76.9)
-		(end 102.639339 77.046446)
-		(width 0.15)
-		(layer "In1.Cu")
-		(net 42)
-	)
-	(segment
-		(start 102.639339 77.046446)
+		(start 94.603554 77.046446)
 		(end 104.053554 77.046446)
 		(width 0.15)
@@
 	)
 	(segment
-		(start 91.6 80.05)
-		(end 94.75 76.9)
+		(start 91.6 82.3)
+		(end 91.6 80.05)
 		(width 0.15)
 		(layer "In1.Cu")
@@
 	)
 	(segment
-		(start 94.75 76.9)
-		(end 102.492893 76.9)
+		(start 91.6 80.05)
+		(end 94.603554 77.046446)
 		(width 0.15)
 		(layer "In1.Cu")
@@
 	)
 	(segment
-		(start 106.192095 77.982905)
-		(end 106.126041 78.048959)
+		(start 95.226041 78.048959)
+		(end 92.5 80.775)
 		(width 0.15)
 		(layer "In1.Cu")
@@
 	)
 	(segment
-		(start 106.126041 78.048959)
-		(end 104.843934 78.048959)
-		(width 0.15)
-		(layer "In1.Cu")
-		(net 43)
-	)
-	(segment
-		(start 94.951041 77.898959)
-		(end 92.5 80.35)
-		(width 0.15)
-		(layer "In1.Cu")
-		(net 43)
-	)
-	(segment
-		(start 92.5 89.05)
-		(end 91.25 90.3)
+		(start 106.192095 77.982905)
+		(end 106.126041 78.048959)
 		(width 0.15)
 		(layer "In1.Cu")
@@
 	)
 	(segment
-		(start 104.693934 77.898959)
-		(end 94.951041 77.898959)
+		(start 92.5 80.775)
+		(end 92.5 89.05)
 		(width 0.15)
 		(layer "In1.Cu")
@@
 	)
 	(segment
-		(start 92.5 80.35)
-		(end 92.5 89.05)
+		(start 106.126041 78.048959)
+		(end 95.226041 78.048959)
 		(width 0.15)
 		(layer "In1.Cu")
@@
 	)
 	(segment
-		(start 104.843934 78.048959)
-		(end 104.693934 77.898959)
+		(start 92.5 89.05)
+		(end 91.25 90.3)
 		(width 0.15)
 		(layer "In1.Cu")
@@
 	)
 	(segment
-		(start 113.55 85.4)
-		(end 128.85 100.7)
+		(start 113.189773 77.860227)
+		(end 113.45 78.120454)
 		(width 0.15)
 		(layer "In1.Cu")
@@
 	)
 	(segment
-		(start 151.35 100.7)
-		(end 156.65 95.4)
+		(start 128.85 100.7)
+		(end 151.35 100.7)
 		(width 0.15)
 		(layer "In1.Cu")
@@
 	)
 	(segment
-		(start 113.55 78.220454)
-		(end 113.55 85.4)
+		(start 151.35 100.7)
+		(end 156.65 95.4)
 		(width 0.15)
 		(layer "In1.Cu")
@@
 	)
 	(segment
-		(start 128.85 100.7)
-		(end 151.35 100.7)
+		(start 113.45 78.120454)
+		(end 113.45 85.3)
 		(width 0.15)
 		(layer "In1.Cu")
@@
 	)
 	(segment
-		(start 113.189773 77.860227)
-		(end 113.55 78.220454)
+		(start 113.45 85.3)
+		(end 128.85 100.7)
 		(width 0.15)
 		(layer "In1.Cu")
