File: photon_bldc/hardware/pcb/one_sided_main_board/main_board.kicad_pcb (KiCad board)
At the start: 4 copper layers, 100 x 64 mm, 46 parts, among them J1 -VIN+, J2 Micro_SD_Card, J3 Conn_01x18, SW2 SW_SPST, U1 STM32G474RETx, U2 AMS1117-5.0, U3 AMS1117-3.3, U5 SST25VF080B-50-4x-S2Ax, X1 24Mhz, X2 32.768KHz

Commit message: kjklj
Parts:
- added D2: BLUE, LED_SMD:LED_0603_1608Metric, F.Cu at (115.3, 55.7)
- added R2: 510R, Resistor_SMD:R_0603_1608Metric, F.Cu at (111.3, 58.4)
- moved PWMR1 94.9 mm to (181.8, 90.5), turned to 90 degrees
- moved PWMT1 94.7 mm to (88.0, 75.9), turned to -90 degrees
- moved R1 41.9 mm to (158.3, 58.3), turned to 0 degrees
- moved D1 35.5 mm to (154.8, 55.8)
- moved R5 8.49 mm to (121.3, 94.1)
- moved R6 8.43 mm to (118.1, 94.0)
- moved J1 6.51 mm to (169.1, 101.9), turned to -90 degrees
- moved C8 2.58 mm to (112.0, 82.2), turned to 0 degrees
- moved C6 2.22 mm to (98.9, 69.8), turned to 180 degrees
- moved U6 2.06 mm to (164.5, 92.0)
- moved J2 1.90 mm to (102.9, 104.9)
- moved L1 1.60 mm to (96.7, 80.6)
- moved C10 1.55 mm to (95.2, 80.6)
- moved Encoder_L1 0.81 mm to (88.0, 88.8)
- moved J3 0.74 mm to (135.0, 49.2)
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Connections:
- U1 pad 2: LED_ON -> LEDON
Routing:
- net VDC: track 0.00 -> 156.9 mm
- net UART1_TX: track 0.00 -> 94.4 mm, vias 0 -> 2
- net UART1_RX: track 0.00 -> 92.7 mm, vias 0 -> 2
- net SPI3_INT: track 0.00 -> 86.5 mm, vias 0 -> 2
- net ENC_R_B: track 0.00 -> 86.1 mm, vias 0 -> 2
- net PWM_R: track 0.00 -> 85.2 mm, vias 0 -> 2
- net ENC_R_A: track 0.00 -> 83.7 mm, vias 0 -> 2
- net SPI3_CS: track 0.00 -> 73.9 mm, vias 0 -> 2
- net SPI3_SCL: track 0.00 -> 71.4 mm, vias 0 -> 2
- net SPI3_MOSI: track 0.00 -> 68.7 mm, vias 0 -> 2
- net LED_1: track 0.00 -> 68.1 mm, vias 0 -> 2
- net SPI3_MISO: track 0.00 -> 64.8 mm, vias 0 -> 2
- net +3.3V: track 0.00 -> 61.2 mm, vias 0 -> 19
- net LEDON: track 0.00 -> 50.3 mm
- net Sensor12: track 0.00 -> 48.1 mm, vias 0 -> 2
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- added copper zone on In1.Cu, net +3.3V
- added copper zone on In2.Cu, net +5V
- added copper zone on B.Cu, net GND
- added copper zone on F.Cu, net GND
Other:
- board text added: "HC-04"

Commit message: 11.05.2025r
Parts:
- added G***: LOGO, LOGO, F.Cu at (137.6, 107.3)
- added G***: LOGO, LOGO, F.Cu at (123.7, 106.5)
- moved C4 4.52 mm to (103.8, 66.6), turned to -90 degrees
- moved C3 2.59 mm to (108.3, 67.0), turned to 90 degrees
- moved X1 2.09 mm to (106.1, 66.8), turned to 0 degrees
- moved C5 1.45 mm to (111.2, 70.0)
- moved C9 1.40 mm to (112.9, 73.3)
- moved C8 1.11 mm to (110.8, 82.3)
- renumbered JP1 to LEDON
Connections:
- J2 pad SH: (no net) -> GND
- J3 pad MP: (no net) -> GND
Routing:
- net GND: track 37.3 -> 27.6 mm, vias 22 -> 23
- net /HSE_OUT: track 10.1 -> 5.01 mm
- net NRST: track 38.4 -> 40.6 mm
- net VREF+: track 8.51 -> 6.59 mm
- net LED_1: track 68.1 -> 69.3 mm
- net SPI2_CLK: track 26.0 -> 27.1 mm
- net SPI2_MISO: track 25.2 -> 26.0 mm
- net /HSE_IN: track 5.24 -> 6.00 mm
- net Net-(D1-A): track 4.50 -> 5.04 mm
- net UART1_RX: track 92.7 -> 93.2 mm
- net +3.3V: track 61.2 -> 60.7 mm, vias 19 -> 21
Other:
- board text added: "+ -"
- board text added: "+3.3V"
- board text added: "+5V"
- board text added: "- ++ -"
- board text added: "CS"
- board text added: "ENCODER L"
- board text added: "ENCODER R"
- board text added: "GND"
- board text added: "INT"
- board text added: "LEDON"
- board text added: "MISO"
- board text added: "MOSI"
- board text added: "PWM L"
- board text added: "PWM R"
- board text added: "PWM T"
- board text added: "SCL"
- board text added: "VIN"

Commit message: 12.05.2025r
Parts:
- moved C7 1.17 mm to (95.8, 67.5), turned to 180 degrees
Routing:
- net PWM_R: track 85.2 -> 169.7 mm
- net NRST: track 40.6 -> 38.4 mm
