File: photon_bldc/hardware/pcb/one_sided_main_board/main_board.kicad_sch (KiCad schematic)
At the start: 46 parts, among them J1 -VIN+, J2 Micro_SD_Card, J3 Conn_01x18, SW2 SW_SPST, U1 STM32G474RETx, U2 AMS1117-5.0, U3 AMS1117-3.3, U5 SST25VF080B-50-4x-S2Ax, X1 24Mhz, X2 32.768KHz

Commit message: kjklj
Parts:
- added D2: BLUE, LED_SMD:LED_0603_1608Metric, symbol Device:LED_Small
- added R2: 510R, Resistor_SMD:R_0603_1608Metric, symbol Device:R
Connections:
- net LED_ON is gone; now on net LEDON: U1.2 (PC13)
- net GND: now also D2.1 (K)
- net LED_2: now also R2.2
- new net: D2.2 (A), R2.1
- no-connect marks 15 -> 16

Commit message: esc
Parts:
- R5: value 1k -> 33k
- R6: value 250R -> 10k
Other:
- note removed: "max 3,186V"
Changed lines of the file:
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@@
-		)
-	)
-	(text "max 3,186V"
-		(exclude_from_sim no)
-		(at 242.57 96.52 0)
-		(effects
-			(font
-				(size 1.1 1.1)
-			)
-			(justify left bottom)
 		)
 	)
@@
 			)
 		)
-		(property "Value" "250R"
+		(property "Value" "10k"
 			(at 237.236 103.378 0)
 			(effects
@@
 			)
 		)
-		(property "Value" "1k"
+		(property "Value" "33k"
 			(at 237.236 93.472 0)
 			(effects
