File: photon_bldc/hardware/pcb/JLCPCB_Order/IMUs/IMU_PCBs/IMU_PCBs.kicad_pcb (KiCad board)
At the start: 2 copper layers, 35.5 x 43.1 mm, 32 parts, among them J1 Conn_01x04, J2 Conn_01x02, U1 ICM-42688-P

Commit message: JJK
Parts:
- added C1: 100n, Capacitor_SMD:C_0402_1005Metric_Pad0.74x0.62mm_HandSolder, F.Cu at (77.6, 111.5)
- added C2: 100n, Capacitor_SMD:C_0402_1005Metric_Pad0.74x0.62mm_HandSolder, F.Cu at (78.6, 111.5)
- added G***: LOGO, LOGO, F.Cu at (80.5, 105.3)
- added G***: LOGO, LOGO, B.Cu at (77.9, 105.6)
- added J1: Conn_01x18, Connector_FFC-FPC:Hirose_FH12-18S-0.5SH_1x18-1MP_P0.50mm_Horizontal, F.Cu at (75.7, 105.6)
- added R1: 47R, Resistor_SMD:R_0603_1608Metric_Pad0.98x0.95mm_HandSolder, B.Cu at (78.0, 58.2)
- added R10: 10K, Resistor_SMD:R_0402_1005Metric_Pad0.72x0.64mm_HandSolder, F.Cu at (83.6, 112.6)
- added R11: 47R, Resistor_SMD:R_0603_1608Metric_Pad0.98x0.95mm_HandSolder, B.Cu at (83.2, 134.2)
- added R12: 10K, Resistor_SMD:R_0402_1005Metric_Pad0.72x0.64mm_HandSolder, F.Cu at (83.5, 136.8)
- added R13: 10K, Resistor_SMD:R_0402_1005Metric_Pad0.72x0.64mm_HandSolder, F.Cu at (80.1, 65.1)
- added R14: 10K, Resistor_SMD:R_0402_1005Metric_Pad0.72x0.64mm_HandSolder, F.Cu at (76.6, 55.6)
- added R15: 10K, Resistor_SMD:R_0402_1005Metric_Pad0.72x0.64mm_HandSolder, F.Cu at (83.6, 131.7)
- added R16: 47R, Resistor_SMD:R_0603_1608Metric_Pad0.98x0.95mm_HandSolder, B.Cu at (78.2, 153.3)
- added R17: 10K, Resistor_SMD:R_0402_1005Metric_Pad0.72x0.64mm_HandSolder, F.Cu at (76.8, 155.8)
- added R18: 10K, Resistor_SMD:R_0402_1005Metric_Pad0.72x0.64mm_HandSolder, F.Cu at (80.2, 146.3)
- added R2: 47R, Resistor_SMD:R_0603_1608Metric_Pad0.98x0.95mm_HandSolder, B.Cu at (83.1, 77.2)
- added R3: 10K, Resistor_SMD:R_0402_1005Metric_Pad0.72x0.64mm_HandSolder, F.Cu at (83.6, 84.1)
- added R4: 10K, Resistor_SMD:R_0402_1005Metric_Pad0.72x0.64mm_HandSolder, F.Cu at (83.6, 74.6)
- added R5: 47R, Resistor_SMD:R_0603_1608Metric_Pad0.98x0.95mm_HandSolder, B.Cu at (83.1, 96.2)
- added R6: 10K, Resistor_SMD:R_0402_1005Metric_Pad0.72x0.64mm_HandSolder, F.Cu at (83.5, 103.1)
- added R7: 10K, Resistor_SMD:R_0402_1005Metric_Pad0.72x0.64mm_HandSolder, F.Cu at (83.6, 93.7)
- added R8: 47R, Resistor_SMD:R_0603_1608Metric_Pad0.98x0.95mm_HandSolder, B.Cu at (83.1, 115.3)
- added R9: 10K, Resistor_SMD:R_0402_1005Metric_Pad0.72x0.64mm_HandSolder, F.Cu at (83.5, 122.2)
- added REF**: MountingHole_2.2mm_M2, MountingHole:MountingHole_2.2mm_M2, F.Cu at (71.5, 44.2)
- added REF**: MountingHole_2.2mm_M2, MountingHole:MountingHole_2.2mm_M2, F.Cu at (71.5, 167.2)
- added U1: ~, SensorOptical:KTIR0711S, B.Cu at (75.0, 53.5)
- added U10: ~, SensorOptical:KTIR0711S, B.Cu at (82.0, 139.0)
- added U11: ~, SensorOptical:KTIR0711S, B.Cu at (78.5, 148.5)
- added U12: ~, SensorOptical:KTIR0711S, B.Cu at (75.0, 158.0)
- added U2: ~, SensorOptical:KTIR0711S, B.Cu at (78.5, 63.0)
- added U3: ~, SensorOptical:KTIR0711S, B.Cu at (82.0, 72.5)
- added U4: ~, SensorOptical:KTIR0711S, B.Cu at (82.0, 82.0)
- added U5: ~, SensorOptical:KTIR0711S, B.Cu at (82.0, 91.5)
- added U6: ~, SensorOptical:KTIR0711S, B.Cu at (82.0, 101.0)
- added U7: ~, SensorOptical:KTIR0711S, B.Cu at (82.0, 110.5)
- added U8: ~, SensorOptical:KTIR0711S, B.Cu at (82.0, 120.0)
- added U9: ~, SensorOptical:KTIR0711S, B.Cu at (82.0, 129.5)
- added mouse-bite-2.54mm-4.66mm: VAL**, mouse-bite:mouse-bite-2.54mm-4.66mm, F.Cu at (87.3, 91.3)
- added mouse-bite-2.54mm-4.66mm: VAL**, mouse-bite:mouse-bite-2.54mm-4.66mm, F.Cu at (87.3, 120.2)
- moved C1 38.5 mm to (102.1, 105.6)
- moved C1 38.5 mm to (110.1, 95.7)
- moved C2 38.5 mm to (101.6, 93.1)
- moved C3 38.5 mm to (110.5, 108.8)
- moved J1 38.5 mm to (110.3, 100.5)
- moved REF** 38.5 mm to (92.1, 87.6)
- moved REF** 38.5 mm to (120.1, 87.6)
- moved U1 38.5 mm to (106.1, 93.3)
- moved U2 38.5 mm to (113.1, 92.1)
- moved C1 38.5 mm to (103.6, 118.5)
- moved C2 38.5 mm to (110.5, 105.7)
- moved C2 38.5 mm to (102.1, 118.5)
- moved C5 38.5 mm to (114.5, 95.2)
- moved D1 38.5 mm to (114.5, 96.8)
- moved IMU_Conn1 38.5 mm to (106.5, 122.3)
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Routing:
- net (no net): track 0.00 -> 418.1 mm, vias 0 -> 12
- net +3.3V: track 51.6 -> 77.3 mm, vias 6 -> 17
- net GND: vias 16 -> 44
Other:
- board size 35.5 x 43.1 mm -> 56.3 x 131.7 mm
- board text added: "1"
- board text added: "10"
- board text added: "11"
- board text added: "12"
- board text added: "2"
- board text added: "3"
- board text added: "4"
- board text added: "5"
- board text added: "6"
- board text added: "7"
- board text added: "8"
- board text added: "9"
- board text added: "S.NYDEREK & P.HELIOS 2025r"
