File: photon_bldc/hardware/pcb/IMU_ICM42688/ICM42688/ICM42688.kicad_pcb (KiCad board)
At the start: 2 copper layers, 11 x 11 mm, 6 parts, among them J1 Conn_01x04, J2 Conn_01x02, U1 ICM-42688-P

Commit message: jgguighuugi
Connections:
- J1 pad 1: SPI_CS -> INT1
- U1 pad 12: SPI_CS -> GND
- U1 pad 4: unconnected-(U1-INT1/INT-Pad4) -> INT1
Routing:
- net INT1: track 0.00 -> 10.1 mm, vias 0 -> 2
- net SPI_CS: track 4.50 -> 0.00 mm
Changed lines of the file:
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@@
 			(outputformat 1)
 			(mirror no)
-			(drillshape 1)
+			(drillshape 0)
 			(scaleselection 1)
-			(outputdirectory "")
+			(outputdirectory "../GERBERS/")
 		)
 	)
@@
 	(net 1 "+3.3V")
 	(net 2 "GND")
-	(net 3 "SPI_CS")
+	(net 3 "INT1")
 	(net 4 "SPI_SCK")
 	(net 5 "SPI_MOSI")
@@
 	(net 8 "unconnected-(U1-RESV_3-Pad3)")
 	(net 9 "unconnected-(U1-RESV_2-Pad2)")
-	(net 10 "unconnected-(U1-INT1{slash}INT-Pad4)")
-	(net 11 "unconnected-(U1-RESV_10-Pad10)")
+	(net 10 "unconnected-(U1-RESV_10-Pad10)")
 	(footprint "Capacitor_SMD:C_0603_1608Metric"
 		(layer "F.Cu")
@@
 				(font
 					(size 1 1)
-					(thickness 0.15)
+					(thickness 0.16)
 				)
 			)
@@
 			(net 9 "unconnected-(U1-RESV_2-Pad2)")
 			(pinfunction "RESV_2")
-			(pintype "passive")
+			(pintype "passive+no_connect")
 		)
 		(pad "3" smd roundrect
@@
 			(net 8 "unconnected-(U1-RESV_3-Pad3)")
 			(pinfunction "RESV_3")
-			(pintype "passive")
+			(pintype "passive+no_connect")
 		)
 		(pad "4" smd roundrect
@@
 			(layers "F.Cu" "F.Paste")
 			(roundrect_rratio 0.25)
-			(net 10 "unconnected-(U1-INT1{slash}INT-Pad4)")
+			(net 3 "INT1")
 			(pinfunction "INT1/INT")
 			(pintype "output")
@@
 			(net 7 "unconnected-(U1-INT2{slash}FSYNC{slash}CLKIN-Pad9)")
 			(pinfunction "INT2/FSYNC/CLKIN")
-			(pintype "bidirectional")
+			(pintype "bidirectional+no_connect")
 		)
 		(pad "10" smd roundrect
@@
 			(layers "F.Cu" "F.Paste")
 			(roundrect_rratio 0.25)
-			(net 11 "unconnected-(U1-RESV_10-Pad10)")
+			(net 10 "unconnected-(U1-RESV_10-Pad10)")
 			(pinfunction "RESV_10")
-			(pintype "passive")
+			(pintype "passive+no_connect")
 		)
 		(pad "11" smd roundrect
@@
 			(layers "F.Cu" "F.Paste")
 			(roundrect_rratio 0.25)
-			(net 3 "SPI_CS")
+			(net 2 "GND")
 			(pinfunction "AP_CS")
 			(pintype "input")
@@
 			(pinfunction "AP_SDA/AP_SDIO/AP_SDI")
 			(pintype "bidirectional")
+		)
+		(model "${KIPRJMOD}/ICM-42688-P/ICM-42688-P.step"
+			(offset
+				(xyz 0 0 0)
+			)
+			(scale
+				(xyz 1 1 1)
+			)
+			(rotate
+				(xyz -90 0 0)
+			)
 		)
 	)
@@
 			(layers "F.Cu" "F.Paste" "F.Mask")
 			(roundrect_rratio 0.25)
-			(net 3 "SPI_CS")
+			(net 3 "INT1")
 			(pinfunction "Pin_1")
 			(pintype "passive")
@@
 				(font
 					(size 1 1)
-					(thickness 0.15)
+					(thickness 0.16)
 				)
 			)
@@
 				(font
 					(size 1 1)
-					(thickness 0.15)
+					(thickness 0.16)
 				)
 			)
@@
 	)
 	(segment
+		(start 140.3 111.560432)
+		(end 140.3 111.2)
+		(width 0.2)
+		(layer "F.Cu")
+		(net 3)
+	)
+	(segment
 		(start 145.95 107.65)
 		(end 145.95 107.425)
@@
 	)
 	(segment
-		(start 143.2 110.4)
-		(end 145.95 107.65)
-		(width 0.15)
+		(start 141.535 112.45)
+		(end 141.189568 112.45)
+		(width 0.2)
 		(layer "F.Cu")
 		(net 3)
 	)
 	(segment
-		(start 143.2 110.785)
-		(end 143.2 110.4)
-		(width 0.15)
-		(layer "F.Cu")
+		(start 141.189568 112.45)
+		(end 140.3 111.560432)
+		(width 0.2)
+		(layer "F.Cu")
+		(net 3)
+	)
+	(segment
+		(start 145.95 108.05)
+		(end 145.95 107.7)
+		(width 0.2)
+		(layer "F.Cu")
+		(net 3)
+	)
+	(segment
+		(start 144.7 109.3)
+		(end 145.95 108.05)
+		(width 0.2)
+		(layer "F.Cu")
+		(net 3)
+	)
+	(via
+		(at 144.7 109.3)
+		(size 0.6)
+		(drill 0.26)
+		(layers "F.Cu" "B.Cu")
+		(net 3)
+	)
+	(via
+		(at 140.3 111.2)
+		(size 0.6)
+		(drill 0.26)
+		(layers "F.Cu" "B.Cu")
+		(net 3)
+	)
+	(segment
+		(start 140.3 110.2)
+		(end 140.7 109.8)
+		(width 0.2)
+		(layer "B.Cu")
+		(net 3)
+	)
+	(segment
+		(start 144.3 109.7)
+		(end 144.7 109.3)
+		(width 0.2)
+		(layer "B.Cu")
+		(net 3)
+	)
+	(segment
+		(start 140.3 111.2)
+		(end 140.3 110.2)
+		(width 0.2)
+		(layer "B.Cu")
+		(net 3)
+	)
+	(segment
+		(start 140.7 109.8)
+		(end 140.8 109.7)
+		(width 0.2)
+		(layer "B.Cu")
+		(net 3)
+	)
+	(segment
+		(start 140.8 109.7)
+		(end 144.3 109.7)
+		(width 0.2)
+		(layer "B.Cu")
 		(net 3)
 	)
@@
 		(polygon
 			(pts
-				(xy 142 111.2) (xy 143.4 111.2) (xy 143.4 112.2) (xy 142 112.2)
-			)
-		)
+				(xy 142.05 111.25) (xy 143.35 111.25) (xy 143.35 112.15) (xy 142.05 112.15)
+			)
+		)

Commit message: 6.05.25
Parts:
- removed J2: Conn_01x02, Connector:2_cable_pad
- added J3: Conn_01x03, Connector:3_cable_pad, F.Cu at (139.7, 117.1)
- moved J1 0.20 mm to (146.8, 106.3)
Connections:
- J1 pad 1: INT1 -> SPI_CS
- U1 pad 12: GND -> SPI_CS
Routing:
- net INT1: track 10.1 -> 3.58 mm, vias 2 -> 0
- net SPI_CS: track 0.00 -> 4.45 mm
- net +3.3V: track 17.2 -> 16.7 mm, vias 0 -> 2

Commit message: SDFSDFSDF
Parts:
- C1, C2, C3: footprint Capacitor_SMD:C_0603_1608Metric -> Capacitor_SMD:C_0402_1005Metric_Pad0.74x0.62mm_HandSolder
- moved C3 4.67 mm to (144.7, 110.7)
- moved J3 2.17 mm to (138.7, 115.2)
- moved C2 1.64 mm to (145.6, 110.7), turned to -90 degrees
- moved U1 1.41 mm to (141.7, 110.7)
- moved C1 1.16 mm to (138.1, 110.6)
- moved J1 0.98 mm to (145.8, 106.2)
Routing:
- net GND: track 0.00 -> 3.23 mm
- net +3.3V: track 16.7 -> 14.0 mm
- net SPI_MISO: track 4.77 -> 3.33 mm
- net SPI_MOSI: track 3.63 -> 2.35 mm
- net SPI_SCK: track 3.79 -> 2.54 mm
- net INT1: track 3.58 -> 2.89 mm
Other:
- board size 11 x 11 mm -> 9 x 9 mm
- board text added: "GYAT"
