File: photon_bldc/hardware/pcb/G071_ESC_rev2/ESC_PCB/ESC_PCB.kicad_pcb (KiCad board)
At the start: 6 copper layers, 19 x 42 mm, 63 parts, among them J2 Plus, J3 Minus, Q1 NMOS, Q2 NMOS, Q3 NMOS, Q4 NMOS, Q5 NMOS, Q6 NMOS, U1 STM32G071GBUx, U4 L78L06_SOT89

Commit message: FINIIIISZZZ
Parts:
- R10, R5, R6, R7, R8, R9: footprint Resistor_SMD:R_0201_0603Metric_Pad0.64x0.40mm_HandSolder -> Resistor_SMD:R_0402_1005Metric_Pad0.72x0.64mm_HandSolder; moved to B.Cu
- moved R10 23.0 mm to (150.6, 85.8), turned to 90 degrees
- moved R8 22.5 mm to (152.6, 85.8), turned to -90 degrees
- moved R9 20.7 mm to (151.6, 85.8), turned to 90 degrees
- moved R5 19.4 mm to (146.2, 82.5)
- moved R6 18.8 mm to (146.1, 83.5), turned to 180 degrees
- moved R7 18.2 mm to (146.1, 84.6), turned to 180 degrees
- moved C12 0.15 mm to (145.6, 74.2)
- moved TP4 0.15 mm to (154.7, 79.2)
- moved TP9 0.15 mm to (156.3, 49.4)
- moved TP3 0.10 mm to (154.7, 77.2)
- moved TP2 0.05 mm to (154.7, 75.2)
- moved TP10 0.05 mm to (149.7, 49.4)
- moved TP11 0.05 mm to (142.7, 49.4)
Routing:
- net PHASE_B: track 0.00 -> 33.4 mm, vias 33 -> 34
- net PHASE_C: track 0.00 -> 22.3 mm, vias 29 -> 27
- net BEMF_C: track 1.90 -> 11.7 mm
- net BEMF_B: track 1.26 -> 11.0 mm, vias 0 -> 2
- net BEMF_REF: track 24.4 -> 34.0 mm
- net +6V: track 15.4 -> 19.6 mm, vias 6 -> 5
- net Net-(D3-K): track 3.58 -> 4.87 mm
- net INPUT: track 15.1 -> 14.2 mm
- net GND: track 43.9 -> 43.2 mm, vias 115 -> 114
- net +3.3V: track 9.68 -> 9.38 mm, vias 4 -> 3
- net VDC: vias 115 -> 111
Other:
- board text added: "+"
- board text added: "-"
- board text added: "27.07.2025"
- board text added: "GYAT"
- board text added: "S"
- board text added: "Szymon Nyderek Piotr Helios"

Commit message: thrsthj
Connections:
- C2 pad 1: VDC -> +6V
- U2 pad 1: VDC -> +6V
- U2 pad 3: VDC -> +6V
Routing:
- net +6V: track 19.6 -> 27.6 mm
- net VDC: track 15.3 -> 9.37 mm
