File: photon_bldc/hardware/pcb/Encoder_KTH_7812/KTH7812/KTH7812.kicad_sch (KiCad schematic)
At the start: 1 part

Commit message: ikik
Parts:
- added C1: 100n, Capacitor_SMD:C_0402_1005Metric, symbol Device:C
- added TP1, TP2, TP3, TP4, TP5: TestPoint, TestPoint:TestPoint_Pad_1.0x1.0mm, symbol Connector:TestPoint
- U1: footprint (none) -> Library:KTH7812
Connections:
- net +3.3V: now also U1.4 (MOSI), U1.5 (CS), C1.1, TP1.1; no longer U1.13 (VDD)
- net A: now also TP4.1
- net B: now also TP3.1
- net GND: now also TP2.1
- net Z: now reaches U1.3 (Z)
- net Z: now also TP5.1
- new net: C1.2, U1.13 (VDD)
- no-connect marks 0 -> 7
